File: PCB/CANBUS_USB.brd (EAGLE design)
At the start: 63.5 x 69.5 mm, 22 parts

Commit message: CAN Bus
Routing:
- net VCC_MCU: track 59.0 -> 78.6 mm, vias 0 -> 2
Changed lines of the file:
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@@
 <wire x1="47.1768" y1="64.8681" x2="47.1768" y2="62.1876" width="0.1524" layer="1"/>
 <wire x1="46.8194" y1="58.4349" x2="46.86" y2="58.42" width="0.1524" layer="1"/>
-<wire x1="47.1768" y1="64.8681" x2="47.26" y2="64.88" width="0.1524" layer="1"/>
 <wire x1="11.9729" y1="64.1533" x2="11.6155" y2="64.1533" width="0.1524" layer="1"/>
 <wire x1="12.509" y1="64.6894" x2="11.9729" y2="64.1533" width="0.1524" layer="1"/>
@@
 <contactref element="C2" pad="2"/>
 <contactref element="U$1" pad="VUSB"/>
-<wire x1="5.5397" y1="62.7237" x2="6.0758" y2="62.7237" width="0.1524" layer="1"/>
-<wire x1="4.1101" y1="61.2941" x2="5.5397" y2="62.7237" width="0.1524" layer="1"/>
-<wire x1="4.1101" y1="56.2905" x2="4.1101" y2="61.2941" width="0.1524" layer="1"/>
-<wire x1="3.7527" y1="55.9331" x2="4.1101" y2="56.2905" width="0.1524" layer="1"/>
-<wire x1="6.0758" y1="62.7237" x2="6.165" y2="62.865" width="0.1524" layer="1"/>
-<wire x1="3.7527" y1="55.9331" x2="3.68" y2="55.88" width="0.1524" layer="1"/>
-<wire x1="11.2581" y1="58.0775" x2="11.2581" y2="55.9331" width="0.1524" layer="1"/>
-<wire x1="6.6119" y1="62.7237" x2="11.2581" y2="58.0775" width="0.1524" layer="1"/>
-<wire x1="6.2545" y1="62.7237" x2="6.6119" y2="62.7237" width="0.1524" layer="1"/>
-<wire x1="11.2581" y1="55.9331" x2="11.3" y2="55.88" width="0.1524" layer="1"/>
-<wire x1="6.2545" y1="62.7237" x2="6.165" y2="62.865" width="0.1524" layer="1"/>
-<wire x1="10.0072" y1="19.4783" x2="10.0072" y2="19.1209" width="0.1524" layer="1"/>
-<wire x1="9.2924" y1="20.1931" x2="10.0072" y2="19.4783" width="0.1524" layer="1"/>
-<wire x1="7.148" y1="20.1931" x2="9.2924" y2="20.1931" width="0.1524" layer="1"/>
-<wire x1="6.9693" y1="20.0144" x2="7.148" y2="20.1931" width="0.1524" layer="1"/>
-<wire x1="6.6119" y1="20.0144" x2="6.9693" y2="20.0144" width="0.1524" layer="1"/>
-<wire x1="4.1101" y1="22.5162" x2="6.6119" y2="20.0144" width="0.1524" layer="1"/>
-<wire x1="4.1101" y1="55.397" x2="4.1101" y2="22.5162" width="0.1524" layer="1"/>
-<wire x1="3.7527" y1="55.7544" x2="4.1101" y2="55.397" width="0.1524" layer="1"/>
-<wire x1="10.0072" y1="19.1209" x2="10.16" y2="19.05" width="0.1524" layer="1"/>
-<wire x1="3.7527" y1="55.7544" x2="3.68" y2="55.88" width="0.1524" layer="1"/>
+<wire x1="6.165" y1="62.865" x2="5.715" y2="62.865" width="1.016" layer="1"/>
+<wire x1="3.68" y1="60.83" x2="3.68" y2="55.88" width="1.016" layer="1"/>
+<wire x1="5.715" y1="62.865" x2="3.68" y2="60.83" width="1.016" layer="1"/>
+<wire x1="3.68" y1="55.88" x2="3.81" y2="55.75" width="1.016" layer="1"/>
+<wire x1="3.81" y1="55.75" x2="3.81" y2="53.34" width="1.016" layer="1"/>
+<wire x1="3.81" y1="53.34" x2="3.81" y2="13.97" width="1.016" layer="1"/>
+<wire x1="3.81" y1="13.97" x2="5.08" y2="12.7" width="1.016" layer="1"/>
+<wire x1="7.62" y1="12.7" x2="11.43" y2="16.51" width="1.016" layer="1"/>
+<wire x1="11.43" y1="16.51" x2="10.16" y2="17.78" width="1.016" layer="1"/>
+<wire x1="10.16" y1="17.78" x2="10.16" y2="19.05" width="1.016" layer="1"/>
+<wire x1="5.08" y1="12.7" x2="7.62" y2="12.7" width="1.016" layer="1"/>
+<wire x1="3.81" y1="53.34" x2="5.08" y2="52.07" width="1.016" layer="1"/>
+<wire x1="5.08" y1="52.07" x2="10.16" y2="52.07" width="1.016" layer="1"/>
+<via x="10.16" y="52.07" extent="1-16" drill="0.35"/>
+<wire x1="10.16" y1="52.07" x2="13.97" y2="52.07" width="1.016" layer="16"/>
+<via x="13.97" y="52.07" extent="1-16" drill="0.35"/>
+<wire x1="11.3" y1="55.88" x2="13.97" y2="53.21" width="1.016" layer="1"/>
+<wire x1="13.97" y1="53.21" x2="13.97" y2="52.07" width="1.016" layer="1"/>
 </signal>
 <signal name="N$2">
