File: PCB/LEDBox.brd (EAGLE design)
At the start: 28 x 28 mm, 12 parts, among them K1 D2F-5

Commit message: CAN Bus
Routing:
- net GND: track 36.7 -> 35.1 mm
Changed lines of the file:
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@@
 <drawing>
 <settings>
-<setting alwaysvectorfont="yes"/>
+<setting alwaysvectorfont="no"/>
 <setting verticaltext="up"/>
 </settings>
@@
 <vertex x="0.5" y="0.2"/>
 </polygon>
-<contactref element="R1" pad="1"/>
 <contactref element="J2" pad="1"/>
 <contactref element="J1" pad="4"/>
@@
 <via x="10.5" y="11" extent="1-16" drill="0.35"/>
 <wire x1="10.5" y1="11" x2="9.5" y2="12" width="0.1524" layer="1"/>
-<wire x1="9.5" y1="12" x2="9.5" y2="13.6" width="0.1524" layer="1"/>
 <wire x1="22.23" y1="12.46" x2="21.7586" y2="12.9314" width="0.1524" layer="1"/>
 <wire x1="21.7586" y1="12.9314" x2="21.23234375" y2="12.9314" width="0.1524" layer="1"/>
@@
 <wire x1="17.8714" y1="21.7486" x2="17.8714" y2="24.4946875" width="0.1524" layer="1"/>
 <wire x1="19.12" y1="20.5" x2="17.8714" y2="21.7486" width="0.1524" layer="1"/>
+<contactref element="R1" pad="1"/>
+<wire x1="19" y1="26.4" x2="21.56" y2="26.86" width="0" layer="19" extent="1-1"/>
+<wire x1="21.78" y1="6.52" x2="22.23" y2="12.46" width="0" layer="19" extent="1-1"/>
+<wire x1="19.25" y1="6.4" x2="21.78" y2="6.52" width="0" layer="19" extent="1-1"/>
+<wire x1="10.75" y1="26.15" x2="17.8714" y2="24.4946875" width="0" layer="19" extent="1-1"/>
+<wire x1="11" y1="6.4" x2="19.25" y2="6.4" width="0" layer="19" extent="1-1"/>
+<wire x1="9.5" y1="13.6" x2="9.5" y2="12" width="0" layer="19" extent="1-1"/>
+<wire x1="2.37" y1="26.77" x2="10.75" y2="26.15" width="0" layer="19" extent="1-1"/>
 </signal>
 <signal name="VCC">
@@
 </signal>
 <signal name="SDIN">
-<contactref element="R1" pad="2"/>
 <contactref element="K1" pad="2"/>
 <contactref element="J2" pad="4"/>
@@
 <wire x1="9.4488" y1="16.3068" x2="8.6868" y2="16.3068" width="0.1524" layer="1"/>
 <wire x1="22.2504" y1="15.3924" x2="22.23" y2="15.46" width="0.1524" layer="1"/>
-<wire x1="9.4488" y1="16.3068" x2="9.5" y2="16.4" width="0.1524" layer="1"/>
 <wire x1="4.572" y1="14.7828" x2="3.5052" y2="14.7828" width="0.1524" layer="1"/>
 <wire x1="4.8768" y1="14.478" x2="4.572" y2="14.7828" width="0.1524" layer="1"/>
 <wire x1="7.9248" y1="14.478" x2="4.8768" y2="14.478" width="0.1524" layer="1"/>
 <wire x1="3.5052" y1="14.7828" x2="3.5" y2="14.92" width="0.1524" layer="1"/>
+<contactref element="R1" pad="2"/>
+<wire x1="9.4488" y1="16.3068" x2="9.5" y2="16.4" width="0" layer="19" extent="1-1"/>
 </signal>
 <signal name="SCL">
