File: Circuit/PCB/teensyMotors.brd (EAGLE design)
At the start: 76.3 x 157.6 mm, 53 parts, among them SW1 219-10, U1 MUX-74HC4067

Commit message: updated main board
Parts:
- removed C3: 0.1uF, adafruit:C1206
- removed INPUT_POWER_2, OUTPUT_POWER: MOLEX4015, MOLEX4015:MOLEX4015
- removed M_C10, M_C8: (no value), adafruit:C1206
- removed M_C11, M_C4, M_C5, M_C6, M_C7, M_C9: 100uf, adafruit:C1206
- removed POWER_LED: LEDFAB1206, fab:LED1206FAB
- added C10, C11, C15, C4, C5, C6, C7, C8, C9: 100uF, SparkFun-Capacitors:PANASONIC_D
- added C12, C13, C14, C16: (no value), microbuilder:1206
- added CAN_RST: 10K, SparkFun-Resistors:1206
- added D1, D2: S2M, s2x_10:DO214AA
- added LED1: (no value), SK6812:LED5050_N
- added POWER_LED_M, POWER_LED_MCU: LEDFAB1206, fab:LED1206FAB
- added POWER_LED_RES1: 500, fab:R1206FAB
- added POWER_M, POWER_MCU: B2P-VH, con-JST VH:B2P-VH
- added S1: (no value), SparkFun-Switches:SWITCH_DPDT_SMD_AYZ0202
- added U$2: (no value), 1zac:VSSOP(8)
- added U$4: (no value), v-reg-2:TO263-3
- C2: value 0.1uF -> (none); device adafruit:C1206 -> microbuilder:1206
- CM_01, CM_02, CM_03, CM_04, CM_05, CM_06, CM_07, CM_08: device SparkFun-Connectors:1X04_SMD_VERTICAL_COMBO -> adafruit:1X04-CLEANBIG
- MOTOR_01, MOTOR_02, MOTOR_03, MOTOR_04, MOTOR_05, MOTOR_06, MOTOR_07, MOTOR_08: value STSPIN220PIN -> DRV8880; device STSPIN220:STSPIN220 -> STSPIN220:DRV8880
- moved CAN_R2 109.4 mm to (31.8, 8.89), turned to 90 degrees
- moved MOTOR_01 48.3 mm to (63.5, 19.1), turned to 90 degrees
- moved MOTOR_02 48.3 mm to (15.2, 19.1), turned to 90 degrees
- moved CAN_LED_R 45.9 mm to (45.7, 110.5)
- moved CM_02 44.7 mm to (19.5, 33.7), turned to 0 degrees
- moved CM_01 36.3 mm to (60.1, 33.7), turned to 0 degrees
- moved CAN_LED 35.8 mm to (45.7, 116.8), turned to 90 degrees
- moved CAN_R3 35.3 mm to (31.8, 151.1), turned to 90 degrees
- moved POWER_LED_RES 30.9 mm to (19.1, 123.2)
- moved TCAN1042 23.4 mm to (50.8, 104.1), turned to 0 degrees
- moved C1 17.0 mm to (35.6, 34.3), turned to 270 degrees
- moved CONN01 16.7 mm to (33.0, 90.2)
- moved CONN02 16.6 mm to (48.5, 90.2)
- moved C2 14.2 mm to (36.8, 104.1), turned to 270 degrees
- moved U$1 10.2 mm to (40.2, 59.2)
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Connections:
- removed net CAN_STB: TCAN1042.8, U$1.32
- new net LED_DEBUG: LED1.4-DIN, U$1.32
- new net N$12: D1.A, D2.A
- new net N$13: LED1.2-DOUT
- new net N$2: C14.2, U$2.VCAPH
- new net N$4: U$2.GDRIVE, U$2.GPD, U$4.1
- new net N$5: C14.1, U$2.VCAPL
- new net N$6: CAN_RST.1, TCAN1042.8
- new net N$7: POWER_LED_MCU.1, POWER_LED_RES1.1
- new net N$9: C12.2, C13.1
- new net REG_5V: C15.+, S1.6, U$2.CATHODE, U$4.4
- new net VCC_5V: C2.1, CONN01.11, LED1.1-VDD, MOTOR_01.FAULT, MOTOR_02.FAULT, MOTOR_03.FAULT, MOTOR_04.FAULT, MOTOR_05.FAULT, MOTOR_06.FAULT, MOTOR_07.FAULT, MOTOR_08.FAULT, POWER_LED_RES1.2, S1.3, U$1.VIN
- net 3.3V: now also C16.1, CONN02.11, TCAN1042.3
- net GND_IN: no longer INPUT_POWER_2.GND_01, INPUT_POWER_2.GND_02
- net GND_M: now also C10.-, C11.-, C4.-, C5.-, C6.-, C7.-, C8.-, C9.-, POWER_LED_M.2, POWER_M.2; no longer MOTOR_01.GND_0, MOTOR_02.GND_0, MOTOR_03.GND_0, MOTOR_04.GND_0, MOTOR_05.GND_0, MOTOR_06.GND_0, MOTOR_07.GND_0, MOTOR_08.GND_0, M_C10.2, M_C11.2, M_C4.2, M_C5.2, M_C6.2, M_C7.2, M_C8.2, M_C9.2, OUTPUT_POWER.GND_01, POWER_LED.2
- net GND_MCU: now also C13.2, C15.-, C16.2, C2.2, CAN_RST.2, D2.C, LED1.3-GND, MOTOR_01.GND_0, MOTOR_02.GND_0, MOTOR_03.GND_0, MOTOR_04.GND_0, MOTOR_05.GND_0, MOTOR_06.GND_0, MOTOR_07.GND_0, MOTOR_08.GND_0, POWER_LED_MCU.2, POWER_MCU.2; no longer C2.1, C3.2, OUTPUT_POWER.GND_02
- net N$1: now also POWER_LED_M.1; no longer POWER_LED.1
- net VCC_IN: no longer INPUT_POWER_2.VCC_01, INPUT_POWER_2.VCC_02
- net VCC_M: now also C10.+, C11.+, C4.+, C5.+, C6.+, C7.+, C8.+, C9.+, MOTOR_01.VM, MOTOR_02.VM, MOTOR_03.VM, MOTOR_04.VM, MOTOR_05.VM, MOTOR_06.VM, MOTOR_07.VM, MOTOR_08.VM, POWER_M.1; no longer MOTOR_01.VCC, MOTOR_02.VCC, MOTOR_03.VCC, MOTOR_04.VCC, MOTOR_05.VCC, MOTOR_06.VCC, MOTOR_07.VCC, MOTOR_08.VCC, M_C10.1, M_C11.1, M_C4.1, M_C5.1, M_C6.1, M_C7.1, M_C8.1, M_C9.1, OUTPUT_POWER.VCC_01
- net VCC_MCU: now also C12.1, D1.C, POWER_MCU.1, U$2.ANODE, U$4.3; no longer C2.2, C3.1, CONN01.11, CONN02.11, OUTPUT_POWER.VCC_02, TCAN1042.3, U$1.VIN
Routing:
- net VCC_5V: track 0.00 -> 377.9 mm, vias 0 -> 3
- net GND_M: track 368.7 -> 1.32 mm
- net I2CM_8: track 196.9 -> 35.8 mm, vias 4 -> 3
- net GND_MCU: track 211.7 -> 61.4 mm, vias 11 -> 9
- net CAN_L: track 344.5 -> 232.9 mm, vias 3 -> 2
- net I2CM_7: track 140.8 -> 30.4 mm, vias 5 -> 1
- net MDIR_03: track 130.4 -> 27.9 mm, vias 7 -> 1
- net CAN_TX: track 220.6 -> 119.2 mm, vias 7 -> 4
- net 3.3V: track 202.0 -> 107.9 mm, vias 10 -> 2
- net CAN_STB: track 82.2 -> 0.00 mm, vias 4 -> 0
- net MDIR_01: track 126.0 -> 55.1 mm
- net MB2_03: track 76.1 -> 9.01 mm, vias 3 -> 0
- net MENABLE: track 335.5 -> 399.4 mm, vias 9 -> 10
- net LED_DEBUG: track 0.00 -> 57.3 mm, vias 0 -> 2
- net REG_5V: track 0.00 -> 48.7 mm
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Other:
- board text added: "CAN"
- board text added: "Debug"
- board text added: "ON"
- board text added: "POWER"
- board text removed: "OUT"
