File: Circuit/PCB/teensyMotors.sch (EAGLE design)
At the start: 53 parts, among them SW1 219-10, U1 MUX-74HC4067

Commit message: updated main board
Parts:
- removed C3: 0.1uF, adafruit:C-USC1206
- removed INPUT_POWER_2, OUTPUT_POWER: MOLEX4015, MOLEX4015:MOLEX4015
- removed M_C10, M_C8: (no value), adafruit:C-USC1206
- removed M_C11, M_C4, M_C5, M_C6, M_C7, M_C9: 100uf, adafruit:C-USC1206
- removed POWER_LED: LEDFAB1206, fab:LEDFAB1206
- added C10, C11, C15, C4, C5, C6, C7, C8, C9: 100uF, SparkFun-Capacitors:100UF-POLAR-25V-20%(ELEC)
- added C12, C13, C14, C16: (no value), microbuilder:CAP_CERAMIC1206
- added CAN_RST: 10K, SparkFun-Resistors:RESISTOR1206
- added D1, D2: S2M, s2x_10:S2M
- added LED1: (no value), SK6812:SK6812_5050N
- added POWER_LED_M, POWER_LED_MCU: LEDFAB1206, fab:LEDFAB1206
- added POWER_LED_RES1: 500, fab:RES-US1206FAB
- added POWER_M, POWER_MCU: B2P-VH, con-JST VH:B2P-VH
- added S1: (no value), SparkFun-Switches:SWITCH-DPDT-SMD-AYZ0202
- added U$2: (no value), 1zac:LM74610-Q1
- added U$4: (no value), v-reg-2:BUK
- C2: value 0.1uF -> (none); device adafruit:C-USC1206 -> microbuilder:CAP_CERAMIC1206
- CM_01, CM_02, CM_03, CM_04, CM_05, CM_06, CM_07, CM_08: device SparkFun-Connectors:CONN_04SMD_STRAIGHT_COMBO -> adafruit:1X4-CLEANBIG
- MOTOR_01, MOTOR_02, MOTOR_03, MOTOR_04, MOTOR_05, MOTOR_06, MOTOR_07, MOTOR_08: value STSPIN220PIN -> DRV8880; device STSPIN220:STSPIN220PIN -> STSPIN220:DRV8880
Connections:
- removed net CAN_STB: TCAN1042.STB, U$1.32/T/PWM
- new net LED_DEBUG: LED1.DI, U$1.32/T/PWM
- new net N$12: D1.A, D2.A
- new net N$13: LED1.DO
- new net N$2: C14.P$2, U$2.VCAPH
- new net N$4: U$2.GDRIVE, U$2.GPD, U$4.IN
- new net N$5: C14.P$1, U$2.VCAPL
- new net N$6: CAN_RST.1, TCAN1042.STB
- new net N$7: POWER_LED_MCU.A, POWER_LED_RES1.1
- new net N$9: C12.P$2, C13.P$1
- new net REG_5V: C15.+, S1.6, U$2.CATHODE, U$4.GND
- new net VCC_5V: C2.P$1, CONN01.11, LED1.VDD, MOTOR_01.FAULT, MOTOR_02.FAULT, MOTOR_03.FAULT, MOTOR_04.FAULT, MOTOR_05.FAULT, MOTOR_06.FAULT, MOTOR_07.FAULT, MOTOR_08.FAULT, POWER_LED_RES1.2, S1.3, U$1.VIN
- net 3.3V: now also C16.P$1, CONN02.11, TCAN1042.VCC
- net GND_IN: no longer INPUT_POWER_2.GND_01, INPUT_POWER_2.GND_02
- net GND_M: now also C10.-, C11.-, C4.-, C5.-, C6.-, C7.-, C8.-, C9.-, POWER_LED_M.C, POWER_M.2; no longer MOTOR_01.GND_0, MOTOR_02.GND_0, MOTOR_03.GND_0, MOTOR_04.GND_0, MOTOR_05.GND_0, MOTOR_06.GND_0, MOTOR_07.GND_0, MOTOR_08.GND_0, M_C10.2, M_C11.2, M_C4.2, M_C5.2, M_C6.2, M_C7.2, M_C8.2, M_C9.2, OUTPUT_POWER.GND_01, POWER_LED.C
- net GND_MCU: now also C13.P$2, C15.-, C16.P$2, C2.P$2, CAN_RST.2, D2.C, LED1.GND, MOTOR_01.GND_0, MOTOR_02.GND_0, MOTOR_03.GND_0, MOTOR_04.GND_0, MOTOR_05.GND_0, MOTOR_06.GND_0, MOTOR_07.GND_0, MOTOR_08.GND_0, POWER_LED_MCU.C, POWER_MCU.2; no longer C2.1, C3.2, OUTPUT_POWER.GND_02
- net N$1: now also POWER_LED_M.A; no longer POWER_LED.A
- net VCC_IN: no longer INPUT_POWER_2.VCC_01, INPUT_POWER_2.VCC_02
- net VCC_M: now also C10.+, C11.+, C4.+, C5.+, C6.+, C7.+, C8.+, C9.+, MOTOR_01.VM, MOTOR_02.VM, MOTOR_03.VM, MOTOR_04.VM, MOTOR_05.VM, MOTOR_06.VM, MOTOR_07.VM, MOTOR_08.VM, POWER_M.1; no longer MOTOR_01.VCC, MOTOR_02.VCC, MOTOR_03.VCC, MOTOR_04.VCC, MOTOR_05.VCC, MOTOR_06.VCC, MOTOR_07.VCC, MOTOR_08.VCC, M_C10.1, M_C11.1, M_C4.1, M_C5.1, M_C6.1, M_C7.1, M_C8.1, M_C9.1, OUTPUT_POWER.VCC_01
- net VCC_MCU: now also C12.P$1, D1.C, POWER_MCU.1, U$2.ANODE, U$4.OUT; no longer C2.2, C3.1, CONN01.11, CONN02.11, OUTPUT_POWER.VCC_02, TCAN1042.VCC, U$1.VIN
Other:
- note added: "REGULATOR"
- moved on the sheet: C2, CM_01, CM_02, CM_03, CM_04, CM_05, CM_06, CM_07, CM_08, POWER_LED_RES
