File: Circuit/PCB/teensyMotors01.brd (EAGLE design)
At the start: 76.3 x 157.6 mm, 66 parts, among them SW1 219-10, U1 MUX-74HC4067

Commit message: clean up
Parts:
- C1, C12, C13, C16, C2: value (none) -> 0.1uf
- C14: value (none) -> 2.2uF
Changed lines of the file:
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@@
 <attribute name="PROD_ID" value="CAP-12547" x="6.35" y="123.19" size="1.778" layer="28" rot="MR180" display="off"/>
 </element>
-<element name="C12" library="microbuilder" package="1206" value="" x="15.24" y="135.89" rot="R270"/>
-<element name="C13" library="microbuilder" package="1206" value="" x="20.32" y="135.89" rot="R90"/>
-<element name="C14" library="microbuilder" package="1206" value="" x="17.78" y="130.81"/>
+<element name="C12" library="microbuilder" package="1206" value="0.1uf" x="15.24" y="135.89" rot="R270"/>
+<element name="C13" library="microbuilder" package="1206" value="0.1uf" x="20.32" y="135.89" rot="R90"/>
+<element name="C14" library="microbuilder" package="1206" value="2.2uF" x="17.78" y="130.81"/>
 <element name="C15" library="SparkFun-Capacitors" library_urn="urn:adsk.eagle:library:510" package="PANASONIC_D" package3d_urn="urn:adsk.eagle:package:37420/1" value="100uF" x="17.78" y="143.51" rot="R270">
 <attribute name="PROD_ID" value="CAP-12547" x="17.78" y="143.51" size="1.778" layer="27" rot="R270" display="off"/>
@@
 </element>
 <element name="U$4" library="v-reg-2" package="TO263-3" value="" x="8.89" y="137.16" rot="R180"/>
-<element name="C16" library="microbuilder" package="1206" value="" x="44.45" y="104.14" rot="R270"/>
+<element name="C16" library="microbuilder" package="1206" value="0.1uf" x="44.45" y="104.14" rot="R270"/>
 <element name="CAN_RST" library="SparkFun-Resistors" library_urn="urn:adsk.eagle:library:532" package="1206" package3d_urn="urn:adsk.eagle:package:39654/1" value="10K" x="40.64" y="104.14" rot="R270">
 <attribute name="PROD_ID" value=" " x="40.64" y="104.14" size="1.778" layer="27" rot="R270" display="off"/>
@@
 <element name="POWER_LED_RES1" library="fab" package="R1206FAB" value="500" x="39.37" y="110.49" rot="R180"/>
 <element name="LED1" library="SK6812" package="LED5050_N" value="" x="30.48" y="104.14"/>
-<element name="C2" library="microbuilder" package="1206" value="" x="36.83" y="104.14" rot="R270"/>
+<element name="C2" library="microbuilder" package="1206" value="0.1uf" x="36.83" y="104.14" rot="R270"/>
 <element name="POWER_M" library="con-JST VH" package="B2P-VH" value="B2P-VH" x="48.26" y="138.43"/>
 <element name="POWER_MCU" library="con-JST VH" package="B2P-VH" value="B2P-VH" x="33.02" y="138.43"/>
-<element name="C1" library="microbuilder" package="1206" value="" x="35.56" y="34.29" rot="R270"/>
+<element name="C1" library="microbuilder" package="1206" value="0.1uf" x="35.56" y="34.29" rot="R270"/>
 </elements>
 <signals>
