File: Circuit/PCB/teensyMotors01.sch (EAGLE design)
At the start: 66 parts, among them SW1 219-10, U1 MUX-74HC4067

Commit message: updated main board
Parts:
- C1: value 0.1uF -> (none); device adafruit:C-USC1206 -> microbuilder:CAP_CERAMIC1206
Connections:
- net 3.3V: now also C1.P$1, CONN02.11; no longer C1.1
- net GND_MCU: now also C1.P$2; no longer C1.2
- net VCC_5V: now also CONN01.11
- net VCC_MCU: no longer CONN01.11, CONN02.11
Changed lines of the file:
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@@
 </variantdefs>
 <classes>
-<class number="0" name="default" width="0" drill="0">
+<class number="0" name="default" width="0.2" drill="0">
 <clearance class="0" value="0.205"/>
+</class>
+<class number="1" name="2oz" width="0.2" drill="0">
 </class>
 </classes>
@@
 <part name="CAN_OUTPUT" library="SparkFun-Connectors" library_urn="urn:adsk.eagle:library:513" deviceset="CONN_02" device="-JST-2MM-SMT" package3d_urn="urn:adsk.eagle:package:38042/1"/>
 <part name="U1" library="SparkFun" deviceset="MUX-74HC4067" device="SMD" value="MUX-74HC4067"/>
-<part name="C1" library="adafruit" deviceset="C-US" device="C1206" value="0.1uF"/>
 <part name="R1" library="SparkFun-Resistors" library_urn="urn:adsk.eagle:library:532" deviceset="RESISTOR" device="1206" package3d_urn="urn:adsk.eagle:package:39654/1" value=" "/>
 <part name="STANDOFF5" library="SparkFun-Electromechanical" library_urn="urn:adsk.eagle:library:516" deviceset="STAND-OFF" device=""/>
@@
 <part name="POWER_M" library="con-JST VH" deviceset="B2P-VH" device="" value="B2P-VH"/>
 <part name="POWER_MCU" library="con-JST VH" deviceset="B2P-VH" device="" value="B2P-VH"/>
+<part name="C1" library="microbuilder" deviceset="CAP_CERAMIC" device="1206"/>
 </parts>
 <sheets>
@@
 <instance part="CAN_OUTPUT" gate="G$1" x="233.68" y="-137.16"/>
 <instance part="U1" gate="G$1" x="-55.88" y="-17.78"/>
-<instance part="C1" gate="G$1" x="-5.08" y="-17.78"/>
 <instance part="R1" gate="G$1" x="-25.4" y="-5.08" rot="R180"/>
 <instance part="STANDOFF5" gate="G$1" x="421.64" y="-101.6"/>
@@
 <instance part="POWER_M" gate="G$1" x="134.62" y="-86.36"/>
 <instance part="POWER_MCU" gate="G$1" x="134.62" y="-104.14"/>
+<instance part="C1" gate="G$1" x="-5.08" y="-20.32"/>
 </instances>
 <busses>
@@
 <pinref part="U1" gate="G$1" pin="VCC"/>
 <wire x1="-5.08" y1="5.08" x2="-5.08" y2="-15.24" width="0.1524" layer="91"/>
-<pinref part="C1" gate="G$1" pin="1"/>
 <wire x1="-35.56" y1="0" x2="-35.56" y2="5.08" width="0.1524" layer="91"/>
 <wire x1="-35.56" y1="5.08" x2="-5.08" y2="5.08" width="0.1524" layer="91"/>
 <junction x="-35.56" y="0"/>
+<pinref part="C1" gate="G$1" pin="P$1"/>
 </segment>
 <segment>
@@
 <pinref part="C16" gate="G$1" pin="P$1"/>
 </segment>
+<segment>
+<pinref part="CONN02" gate="G$1" pin="11"/>
+<wire x1="-132.08" y1="-149.86" x2="-139.7" y2="-149.86" width="0.1524" layer="91"/>
+<label x="-139.7" y="-149.86" size="1.016" layer="95" rot="R180" xref="yes"/>
+</segment>
 </net>
 <net name="I2CM_8" class="0">
@@
 <pinref part="U1" gate="G$1" pin="GND"/>
 <wire x1="-30.48" y1="-33.02" x2="-5.08" y2="-33.02" width="0.1524" layer="91"/>
-<pinref part="C1" gate="G$1" pin="2"/>
 <wire x1="-5.08" y1="-33.02" x2="-5.08" y2="-22.86" width="0.1524" layer="91"/>
 <wire x1="-20.32" y1="-38.1" x2="-30.48" y2="-38.1" width="0.1524" layer="91"/>
 <junction x="-30.48" y="-38.1"/>
+<pinref part="C1" gate="G$1" pin="P$2"/>
 </segment>
 <segment>
@@
 <net name="VCC_MCU" class="0">
 <segment>
-<pinref part="CONN01" gate="G$1" pin="11"/>
-<wire x1="-129.54" y1="-106.68" x2="-137.16" y2="-106.68" width="0.1524" layer="91"/>
-<label x="-137.16" y="-106.68" size="1.016" layer="95" rot="R180" xref="yes"/>
-</segment>
-<segment>
-<pinref part="CONN02" gate="G$1" pin="11"/>
-<wire x1="-132.08" y1="-149.86" x2="-139.7" y2="-149.86" width="0.1524" layer="91"/>
-<label x="-139.7" y="-149.86" size="1.016" layer="95" rot="R180" xref="yes"/>
-</segment>
-<segment>
 <wire x1="408.94" y1="111.76" x2="408.94" y2="66.04" width="0.1524" layer="91"/>
 <pinref part="U$2" gate="G$1" pin="ANODE"/>
@@
 <junction x="441.96" y="-104.14"/>
 </segment>
-</net>
+<segment>
+<pinref part="CONN01" gate="G$1" pin="11"/>
+<wire x1="-129.54" y1="-106.68" x2="-137.16" y2="-106.68" width="0.1524" layer="91"/>
+<label x="-137.16" y="-106.68" size="1.016" layer="95" rot="R180" xref="yes"/>
+</segment>
+</net>

Commit message: clean up
Parts:
- C1, C12, C13, C16, C2: value (none) -> 0.1uf
- C14: value (none) -> 2.2uF
Changed lines of the file:
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@@
 <part name="C10" library="SparkFun-Capacitors" library_urn="urn:adsk.eagle:library:510" deviceset="100UF-POLAR" device="-25V-20%(ELEC)" package3d_urn="urn:adsk.eagle:package:37420/1" value="100uF"/>
 <part name="C11" library="SparkFun-Capacitors" library_urn="urn:adsk.eagle:library:510" deviceset="100UF-POLAR" device="-25V-20%(ELEC)" package3d_urn="urn:adsk.eagle:package:37420/1" value="100uF"/>
-<part name="C12" library="microbuilder" deviceset="CAP_CERAMIC" device="1206"/>
-<part name="C13" library="microbuilder" deviceset="CAP_CERAMIC" device="1206"/>
-<part name="C14" library="microbuilder" deviceset="CAP_CERAMIC" device="1206"/>
+<part name="C12" library="microbuilder" deviceset="CAP_CERAMIC" device="1206" value="0.1uf"/>
+<part name="C13" library="microbuilder" deviceset="CAP_CERAMIC" device="1206" value="0.1uf"/>
+<part name="C14" library="microbuilder" deviceset="CAP_CERAMIC" device="1206" value="2.2uF"/>
 <part name="C15" library="SparkFun-Capacitors" library_urn="urn:adsk.eagle:library:510" deviceset="100UF-POLAR" device="-25V-20%(ELEC)" package3d_urn="urn:adsk.eagle:package:37420/1" value="100uF"/>
 <part name="U$2" library="1zac" deviceset="LM74610-Q1" device=""/>
@@
 <part name="D2" library="s2x_10" deviceset="S2*" device="" technology="M"/>
 <part name="U$4" library="v-reg-2" deviceset="BUK" device=""/>
-<part name="C16" library="microbuilder" deviceset="CAP_CERAMIC" device="1206"/>
+<part name="C16" library="microbuilder" deviceset="CAP_CERAMIC" device="1206" value="0.1uf"/>
 <part name="CAN_RST" library="SparkFun-Resistors" library_urn="urn:adsk.eagle:library:532" deviceset="RESISTOR" device="1206" package3d_urn="urn:adsk.eagle:package:39654/1" value="10K"/>
 <part name="S1" library="SparkFun-Switches" library_urn="urn:adsk.eagle:library:535" deviceset="SWITCH-DPDT" device="-SMD-AYZ0202" package3d_urn="urn:adsk.eagle:package:40160/1">
@@
 <part name="POWER_LED_RES1" library="fab" deviceset="RES-US" device="1206FAB" value="500"/>
 <part name="LED1" library="SK6812" deviceset="SK6812" device="_5050N"/>
-<part name="C2" library="microbuilder" deviceset="CAP_CERAMIC" device="1206"/>
+<part name="C2" library="microbuilder" deviceset="CAP_CERAMIC" device="1206" value="0.1uf"/>
 <part name="POWER_M" library="con-JST VH" deviceset="B2P-VH" device="" value="B2P-VH"/>
 <part name="POWER_MCU" library="con-JST VH" deviceset="B2P-VH" device="" value="B2P-VH"/>
-<part name="C1" library="microbuilder" deviceset="CAP_CERAMIC" device="1206"/>
+<part name="C1" library="microbuilder" deviceset="CAP_CERAMIC" device="1206" value="0.1uf"/>
 </parts>
 <sheets>
