File: Circuit/PCB/teensyMotors02_up.sch (EAGLE design)
At the start: 66 parts, among them SW1 219-10, U1 MUX-74HC4067

Commit message: circuit update
Parts:
- removed C10, C11: 100uF, SparkFun-Capacitors:100UF-POLAR-25V-20%(ELEC)
- removed C12, C13, C16: 0.1uf, microbuilder:CAP_CERAMIC1206
- removed C14: 2.2uF, microbuilder:CAP_CERAMIC1206
- removed CAN_LED, POWER_LED_M, POWER_LED_MCU: LEDFAB1206, fab:LEDFAB1206
- removed CAN_LED_R, POWER_LED_RES, POWER_LED_RES1: 500, fab:RES-US1206FAB
- removed CAN_OUTPUT: (no value), SparkFun-Connectors:CONN_02-JST-2MM-SMT
- removed CAN_R2, CAN_R3: 120ohm, SparkFun-Resistors:RESISTOR1206
- removed CAN_RST: 10K, SparkFun-Resistors:RESISTOR1206
- removed CONN02: TMMH-105-12, TMMH-105-XX-XX-DV:TMMH-105-12
- removed INPUT_POWER_1: MOLEX4015, MOLEX4015:MOLEX4015
- removed J2: (no value), SparkFun-Connectors:CONN_06SMD_MALE
- removed J3, J4: (no value), SparkFun-Connectors:CONN_10SMD_MALE
- removed LED1: (no value), SK6812:SK6812_5050N
- removed STANDOFF5, STANDOFF6, STANDOFF7, STANDOFF8: STAND-OFF, SparkFun-Electromechanical:STAND-OFF
- removed SW1: 219-10, switch-dil:219-10
- removed TCAN1042: Value, TCAN1042DRQ1:TCAN1042DRQ1
- added C3: 0.1uF, SparkFun-Capacitors:0.1UF-25V(+80/-20%)(0603)
- added CAN_INPUT1: (no value), SparkFun-Connectors:CONN_02-JST-2MM-SMT
- added D3: PESD1CAN, diode:PESD1CAN
- added MC1, MC2, MC3, MC4, MC5, MC6, MC7, MC8: 100uF, SparkFun-Capacitors:100UF-POLAR-25V-20%(ELEC)
- added R10: 500, SparkFun-Resistors:10KOHM-1/10W-1%(0603)0603
- added R2, R3, R4, R5, R6, R9: 10K, SparkFun-Resistors:10KOHM-1/10W-1%(0603)0603
- added R7, R8: 60, SparkFun-Resistors:10KOHM-1/10W-1%(0603)0603
- added SJ1: (no value), SparkFun-Passives:JUMPER-PAD-3-NC_BY_TRACE
- added SJ4, SJ5: JUMPER-PAD-3-2OF3_NC_BY_TRACE_SMALL, SparkFun-Passives:JUMPER-PAD-3-2OF3_NC_BY_TRACE_SMALL
- added STATUS_LED: LEDFAB1206, fab:LEDFAB1206
- added U$3: TEENSY_4.0_WITH_SMD_HEADER_PINSTEENSY_4.0_SMD, Teensy4:TEENSY_4.0_WITH_SMD_HEADER_PINSTEENSY_4.0_SMD
- C1, C2: value 0.1uf -> 0.1uF; device microbuilder:CAP_CERAMIC1206 -> SparkFun-Capacitors:0.1UF-25V(+80/-20%)(0603)
- C4, C9: value 100uF -> 2.2uf; device SparkFun-Capacitors:100UF-POLAR-25V-20%(ELEC) -> SparkFun-Capacitors:0.1UF-25V(+80/-20%)(0603)
- C5: value 100uF -> 4.7uf; device SparkFun-Capacitors:100UF-POLAR-25V-20%(ELEC) -> SparkFun-Capacitors:0.1UF-25V(+80/-20%)(0603)
- C6, C7, C8: value 100uF -> 0.1uf; device SparkFun-Capacitors:100UF-POLAR-25V-20%(ELEC) -> SparkFun-Capacitors:0.1UF-25V(+80/-20%)(0603)
- CM_01, CM_02, CM_03, CM_04, CM_05, CM_06, CM_07, CM_08: value 1X04_SMD_STRAIGHT_COMBO -> 1X04_STRAIGHT
- J1: device SparkFun-Connectors:CONN_06SMD_MALE -> SparkFun-Connectors:CONN_02
- R1: value (none) -> 10K; device SparkFun-Resistors:RESISTOR1206 -> SparkFun-Resistors:10KOHM-1/10W-1%(0603)0603
- U$1: value TEENSY_3.1-3.2_ALL_PINS&PADS_SMD -> SN65HVD232Q; device Teensy_3_and_LC_Series_Boards_v1.4:TEENSY_3.1-3.2_ALL_PINS&PADS_SMD -> TCAN1042DRQ1:SN65HVD232Q
- U1: value MUX-74HC4067 -> SX1509; device SparkFun:MUX-74HC4067SMD -> SparkFun-DigitalIC:SX1509
Connections:
- removed net C0: SW1.20, U1.CHAN0
- removed net C1: SW1.19, U1.CHAN1
- removed net C2: SW1.18, U1.CHAN2
- removed net C3: SW1.17, U1.CHAN3
- removed net C4: SW1.16, U1.CHAN4
- removed net C5: SW1.15, U1.CHAN5
- removed net C6: SW1.14, U1.CHAN6
- removed net C7: SW1.13, U1.CHAN7
- removed net C8: SW1.12, U1.CHAN8
- removed net C9: SW1.11, U1.CHAN9
- removed net CAN_RX: TCAN1042.RXD, U$1.4/CAN-RX/PWM
- removed net CAN_TX: CAN_LED_R.2, TCAN1042.TXD, U$1.3/CAN-TX/PWM
- removed net GND_IN: INPUT_POWER_1.GND_01, INPUT_POWER_1.GND_02
- removed net I2CM_0: CONN01.1, J3.9
- removed net I2CM_1: CONN01.2, J3.8
- removed net I2CM_10: CONN02.1, J4.3
- removed net I2CM_11: CONN02.2, J4.4
- removed net I2CM_12: CONN02.3, J4.6
- removed net I2CM_13: CONN02.4, J4.7
- removed net I2CM_14: J4.8
- removed net I2CM_15: CONN02.6, J4.9
- removed net I2CM_2: CONN01.3, J3.7
- removed net I2CM_3: CONN01.4, J3.6
- removed net I2CM_4: CONN01.5, J3.4
- removed net I2CM_5: CONN01.6, J3.3
- removed net I2CM_6: CONN01.7, J3.2
- removed net I2CM_7: CONN01.8, J3.1
- removed net I2CM_8: CONN01.9, J4.1
- removed net I2CM_9: CONN01.10, J4.2
- removed net IC2M_14: CONN02.5
- removed net LED_DEBUG: LED1.DI, U$1.32/T/PWM
- removed net MENABLE: MOTOR_01.ENABLE, MOTOR_02.ENABLE, MOTOR_03.ENABLE, MOTOR_04.ENABLE, MOTOR_05.ENABLE, MOTOR_06.ENABLE, MOTOR_07.ENABLE, MOTOR_08.ENABLE, U$1.33/T
- removed net MUS_S1: U1.S1
- removed net MUX_INT: J1.1
- removed net MUX_OSCIO: J2.1
- removed net MUX_RESET: J1.2, J2.2
- removed net MUX_S0: U$1.26/A15
- removed net MUX_S1: U$1.27/A16
- removed net MUX_S2: U$1.28/A17, U1.S2
- removed net MUX_S3: U$1.31/A20, U1.S3
- removed net MUX_SCL: J1.6, J2.6, U$1.19/A5/T/SCL0
- removed net MUX_SDA: J1.5, J2.5, U$1.18/A4/T/SDA0
- removed net MUX_SIG: U$1.A13, U1.COM
- removed net MUX_SO: U1.S0
- removed net N$11: U$1.13/SCK/LED
- removed net S_SCL: CONN02.10, U$1.29/A18/SCL1
- removed net S_SDA: CONN02.9, U$1.30/A19/SDA1
- removed net S_SEN_01: CONN02.8, U$1.A12
- removed net VCC1: J3.5
- removed net VCC2: J4.5
- removed net VCC_IN: INPUT_POWER_1.VCC_01, INPUT_POWER_1.VCC_02
- new net !INT_SX0: R1.1, U$3.13/SCK/LED, U1.!INT
- new net !RESET_SX0: R3.1, U1.!RESET
- new net 0_SX0: MOTOR_01.ENABLE, U1.I/O[0]
- new net 10_SX0: MOTOR_06.ENABLE, U1.I/O[10]
- new net 11_SX0: MOTOR_06.STBY, U1.I/O[11]
- new net 12_SX0: MOTOR_07.ENABLE, U1.I/O[12]
- new net 13_SX0: MOTOR_07.STBY, U1.I/O[13]
- new net 14_SX0: MOTOR_08.ENABLE, U1.I/O[14]
- new net 15_SX0: MOTOR_08.STBY, U1.I/O[15]
- new net 1_SX0: MOTOR_01.STBY, U1.I/O[1]
- new net 2_SX0: MOTOR_02.ENABLE, U1.I/O[2]
- new net 3_SX0: MOTOR_02.STBY, U1.I/O[3]
- new net 4_SX0: MOTOR_03.ENABLE, U1.I/O[4]
- new net 5_SX0: MOTOR_03.STBY, U1.I/O[5]
- new net 6_SX0: MOTOR_04.ENABLE, U1.I/O[6]
- new net 7_SX0: MOTOR_04.STBY, U1.I/O[7]
- new net 8_SX0: MOTOR_05.ENABLE, U1.I/O[8]
- new net 9_SX0: MOTOR_05.STBY, U1.I/O[9]
- new net ADDR0_SX0: SJ4.2, U1.ADDR0
- new net ADDR1_SX0: SJ5.2, U1.ADDR1
- new net CAN_RX2: CONN01.7, U$3.0/RX1/T/CRX2
- new net CAN_RX3: U$1.RXD, U$3.30/CRX3
- new net CAN_TX2: CONN01.8, U$3.1/TX1/T/CTX2
- new net CAN_TX3: U$1.TXD, U$3.31/CTX3
- new net N$10: R6.1, SJ5.1
- new net N$14: J1.1, R8.1
- new net N$8: R5.1, SJ4.1
- new net OSCIO_SX0: U1.OSCIO
- new net PIN_2: CONN01.6, U$3.2
- new net SCL_00: R2.1, U$3.19/A5/SCL0, U1.SCL
- new net SCL_01: CONN01.1, U$3.16/A2/SCL1
- new net SCL_02: CONN01.3, U$3.24/A10/SCL2
- new net SDA_00: R4.1, U$3.18/A4/SDA0, U1.SDA
- new net SDA_01: CONN01.2, U$3.17/A3/SDA1
- new net SDA_02: CONN01.4, U$3.25/A11/SDA2
- new net STATUS_PIN: R10.2, U$3.4
- new net TRQ1: MOTOR_01.1, MOTOR_02.1, MOTOR_03.1, MOTOR_04.1, MOTOR_05.1, MOTOR_06.1, MOTOR_07.1, MOTOR_08.1, U$3.32
- new net TRQ2: MOTOR_01.2, MOTOR_02.2, MOTOR_03.2, MOTOR_04.2, MOTOR_05.2, MOTOR_06.2, MOTOR_07.2, MOTOR_08.2, U$3.33
- net 3.3V: now also C1.1, C2.1, C3.1, C4.1, C6.1, CONN01.9, R1.2, R3.2, R5.2, R6.2, SJ1.2, U$1.VCC, U$3.3.3V, U1.VCC1, U1.VCC2, U1.VDDM; no longer C1.P$1, C16.P$1, CONN02.11, J1.4, J2.4, TCAN1042.VCC, U$1.3.3V, U1.VCC
- net CAN_H: now also CAN_INPUT1.2, D3.1, R7.2, U$1.CANH; no longer CAN_OUTPUT.2, CAN_R2.1, CAN_R3.1, TCAN1042.CANH
- net CAN_L: now also CAN_INPUT1.1, D3.2, J1.2, U$1.CANL; no longer CAN_OUTPUT.1, CAN_R2.2, CAN_R3.2, TCAN1042.CANL
- net GND_M: now also MC1.-, MC2.-, MC3.-, MC4.-, MC5.-, MC6.-, MC7.-, MC8.-; no longer C10.-, C11.-, C4.-, C5.-, C6.-, C7.-, C8.-, C9.-, POWER_LED_M.C
- net GND_MCU: now also C1.2, C2.2, C3.2, C4.2, C5.2, C6.2, C8.2, CONN01.10, D3.3, R9.2, SJ4.3, SJ5.3, STATUS_LED.C, U$3.GND; no longer C1.P$2, C13.P$2, C16.P$2, C2.P$2, CAN_LED.C, CAN_RST.2, CONN02.12, J1.3, J2.3, LED1.GND, POWER_LED_MCU.C, R1.1, R1.2, SW1.1, SW1.10, SW1.2, SW1.3, SW1.4, SW1.5, SW1.6, SW1.7, SW1.8, SW1.9, TCAN1042.GND, U1.EN
- net MDIR_01: now also U$3.6; no longer U$1.6/PWM
- net MDIR_02: now also U$3.8/TX2; no longer U$1.8/TX3
- net MDIR_03: now also U$3.10/CS; no longer U$1.10/TX2/PWM
- net MDIR_04: now also U$3.12/MISO; no longer U$1.15/A1/T
- net MDIR_05: now also U$3.15/A1/RX3; no longer U$1.17/A3/T
- net MDIR_06: now also U$3.21/A7/RX5; no longer U$1.21/A7/PWM
- net MDIR_07: now also U$3.23/A9/CRX1; no longer U$1.23/A9/T/PWM
- net MDIR_08: now also U$3.27/A13/SCK1; no longer U$1.25/T/PWM
- net MMS1: now also U$3.28/RX7; no longer U$1.11/MOSI
- net MMS2: now also U$3.29/TX7; no longer U$1.12/MISO
- net MSTEP_01: now also U$3.5; no longer U$1.5/PWM
- net MSTEP_02: now also U$3.7/RX2; no longer U$1.7/RX3
- net MSTEP_03: now also U$3.9; no longer U$1.9/RX2/PWM
- net MSTEP_04: now also U$3.11/MOSI; no longer U$1.14/A0
- net MSTEP_05: now also U$3.14/A0/TX3; no longer U$1.16/A2/T
- net MSTEP_06: now also U$3.20/A6/TX5; no longer U$1.20/A6/PWM
- net MSTEP_07: now also U$3.22/A8/CTX1; no longer U$1.22/A8/T/PWM
- net MSTEP_08: now also U$3.26/A12/MOSI1; no longer U$1.24
- net N$1: now also R2.2, SJ1.3; no longer POWER_LED_M.A, POWER_LED_RES.1
- net N$13: now also C5.1, R7.1, R8.2; no longer LED1.DO
- net N$193: now also R10.1, STATUS_LED.A; no longer CAN_LED.A, CAN_LED_R.1
- net N$2: now also C9.1; no longer C14.P$2
- net N$3: now also U$1.NC; no longer TCAN1042.NC
- net N$5: now also C9.2; no longer C14.P$1
- net N$6: now also R9.1, U$1.STB; no longer CAN_RST.1, TCAN1042.STB
- net N$7: now also R4.2, SJ1.1; no longer POWER_LED_MCU.A, POWER_LED_RES1.1
- net N$9: now also C7.2, C8.1; no longer C12.P$2, C13.P$1
- net NEO_PIXEL: now also CONN01.5, U$3.3; no longer CONN02.7, U$1.2
- net VCC_5V: now also S1.2, U$3.VIN; no longer C2.P$1, LED1.VDD, POWER_LED_RES1.2, S1.3, U$1.VIN
- net VCC_M: now also MC1.+, MC2.+, MC3.+, MC4.+, MC5.+, MC6.+, MC7.+, MC8.+; no longer C10.+, C11.+, C4.+, C5.+, C6.+, C7.+, C8.+, C9.+, POWER_LED_RES.2
- net VCC_MCU: now also C7.1; no longer C12.P$1
Other:
- note added: "Allowable VCC1/2 Range: 1.2-3.6V"
- note added: "I2C Address Select"
- note added: "IC2 MUX 01"
- note added: "The VCC1/2 jumpers (SJ2, SJ3) set those pins to 3.3V."
- note added: "VDD Range: 1.425-3.6V"
- note removed: "CONNECTORS"
- note removed: "Control Signal and Power Input Headers"
- note removed: "I/O headers"
- note removed: "I2C MUX"
- note removed: "POWER"
- moved on the sheet: C1, C15, C2, CAN_INPUT, CM_01, CM_02, CM_03, CM_04, CM_05, CM_06, CM_07, CM_08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
