File: Circuit/PCB/teensyMotors02_upSwitch_LED.brd (EAGLE design)
At the start: 72 x 150.1 mm, 80 parts, among them SW1 219-10, U1 SX1509, U2 SX1509, U4 SX1509

Commit message: circuit
Parts:
- removed C1, C2, C3, C4, C5, C6, C7, C8, C9: 0.1uF, SparkFun-Capacitors:0603-CAP
- removed JP10, JP11, JP6, JP7, JP8, JP9: JUMPER-SMT_2_NC_TRACE_NO-SILK, SparkFun-Jumpers:SMT-JUMPER_2_NC_TRACE_NO-SILK
- removed R10, R11, R12, R13, R14, R16, R17, R18, R19, R20, R21, R23, R24, R25, R26, R9: 10K, SparkFun-Resistors:0603-RES
- removed U1, U2, U4: SX1509, SparkFun-DigitalIC:QFN-28
- added U$1, U$2, U$3: SX1509, SX1509_s:SX1509
- moved SW1 41.1 mm to (36.2, 31.0)
- moved R15 40.2 mm to (24.8, 40.0)
- moved R29 40.2 mm to (27.4, 40.0)
- moved R30 40.2 mm to (29.9, 40.0)
- moved R31 40.2 mm to (32.5, 40.0)
- moved R32 40.2 mm to (35.0, 40.0)
- moved R33 40.2 mm to (37.5, 40.0)
- moved R34 40.2 mm to (40.1, 40.0)
- moved R35 40.2 mm to (42.6, 40.0)
- moved R36 40.2 mm to (45.2, 40.0)
- moved R37 40.2 mm to (47.7, 40.0)
- moved S1 25.9 mm to (36.6, 96.0)
Connections:
- removed net !INT_SX1: R12.1, U1.9
- removed net !INT_SX2: R19.1, U2.9
- removed net !INT_SX3: R24.1, U4.9
- removed net !RESET_SX1: R9.1, U1.23
- removed net !RESET_SX2: R16.1, U2.23
- removed net !RESET_SX3: R14.1, U4.23
- removed net ADDR0_SX1: JP8.1, U1.26
- removed net ADDR0_SX2: JP7.1, U2.26
- removed net ADDR0_SX3: JP11.1, U4.26
- removed net ADDR1_SX1: JP9.1, U1.10
- removed net ADDR1_SX2: JP6.1, U2.10
- removed net ADDR1_SX3: JP10.1, U4.10
- removed net N$14: JP10.2, R25.1
- removed net N$15: JP11.2, R26.1
- removed net N$5: JP6.2, R21.1
- removed net N$8: JP8.2, R13.1
- removed net OSCIO_SX1: U1.11
- removed net OSCIO_SX2: U2.11
- removed net OSCIO_SX3: U4.11
- new net N$25: U$3.INT
- new net N$4: U$1.INT
- net 0_SX1: now also U$1.0; no longer U1.27
- net 0_SX2: now also U$2.0; no longer U2.27
- net 0_SX3: now also U$3.0; no longer U4.27
- net 10_SX1: now also U$1.10; no longer U1.15
- net 10_SX2: now also U$2.10; no longer U2.15
- net 10_SX3: now also U$3.10; no longer U4.15
- net 11_SX1: now also U$1.11; no longer U1.16
- net 11_SX2: now also U$2.11; no longer U2.16
- net 11_SX3: now also U$3.11; no longer U4.16
- net 12_SX1: now also U$1.12; no longer U1.19
- net 12_SX2: now also U$2.12; no longer U2.19
- net 12_SX3: now also U$3.12; no longer U4.19
- net 13_SX1: now also U$1.13; no longer U1.20
- net 13_SX2: now also U$2.13; no longer U2.20
- net 13_SX3: now also U$3.13; no longer U4.20
- net 14_SX1: now also U$1.14; no longer U1.21
- net 14_SX2: now also U$2.14; no longer U2.21
- net 14_SX3: now also U$3.14; no longer U4.21
- net 15_SX1: now also U$1.15; no longer U1.22
- net 15_SX2: now also U$2.15; no longer U2.22
- net 15_SX3: now also U$3.15; no longer U4.22
- net 1_SX1: now also U$1.1; no longer U1.28
- net 1_SX2: now also U$2.1; no longer U2.28
- net 1_SX3: now also U$3.1; no longer U4.28
- net 2_SX1: now also U$1.2; no longer U1.1
- net 2_SX2: now also U$2.2; no longer U2.1
- net 2_SX3: now also U$3.2; no longer U4.1
- net 3.3V: now also U$1.3.3V, U$1.3.3V_1, U$2.3.3V, U$2.3.3V_1, U$3.3.3V, U$3.3.3V_1; no longer C1.1, C2.1, C3.1, C4.1, C5.1, C6.1, C7.1, C8.1, C9.1, R10.2, R11.2, R12.2, R13.2, R14.2, R16.2, R17.2, R18.2, R19.2, R20.2, R21.2, R23.2, R24.2, R25.2, R26.2, R9.2, U1.12, U1.18, U1.4, U2.12, U2.18, U2.4, U4.12, U4.18, U4.4
- net 3_SX1: now also U$1.3; no longer U1.2
- net 3_SX2: now also U$2.3; no longer U2.2
- net 3_SX3: now also U$3.3; no longer U4.2
- net 4_SX1: now also U$1.4; no longer U1.5
- net 4_SX2: now also U$2.4; no longer U2.5
- net 4_SX3: now also U$3.4; no longer U4.5
- net 5_SX1: now also U$1.5; no longer U1.6
- net 5_SX2: now also U$2.5; no longer U2.6
- net 5_SX3: now also U$3.5; no longer U4.6
- net 6_SX1: now also U$1.6; no longer U1.7
- net 6_SX2: now also U$2.6; no longer U2.7
- net 6_SX3: now also U$3.6; no longer U4.7
- net 7_SX1: now also U$1.7; no longer U1.8
- net 7_SX2: now also U$2.7; no longer U2.8
- net 7_SX3: now also U$3.7; no longer U4.8
- net 8_SX1: now also U$1.8; no longer U1.13
- net 8_SX2: now also U$2.8; no longer U2.13
- net 8_SX3: now also U$3.8; no longer U4.13
- net 9_SX1: now also U$1.9; no longer U1.14
- net 9_SX2: now also U$2.9; no longer U2.14
- net 9_SX3: now also U$3.9; no longer U4.14
- net GND_MCU: now also U$1.GND, U$1.GND_1, U$1.GND_2, U$1.GND_3, U$2.GND, U$2.GND_1, U$2.GND_2, U$2.GND_3, U$3.GND, U$3.GND_1, U$3.GND_2, U$3.GND_3; no longer C1.2, C2.2, C3.2, C4.2, C5.2, C6.2, C7.2, C8.2, C9.2, JP7.2, JP9.2, U1.17, U1.29, U1.3, U2.17, U2.29, U2.3, U4.17, U4.29, U4.3
- net SCL_00: now also U$1.SCL, U$1.SCL_2, U$1.SDA, U$1.SDA_2, U$2.SCL, U$2.SCL_2, U$3.SCL, U$3.SCL_2; no longer R11.1, R18.1, R23.1, U1.25, U2.25, U4.25
- net SDA_00: now also U$2.SDA, U$2.SDA_2, U$3.SDA, U$3.SDA_2; no longer R10.1, R17.1, R20.1, U1.24, U2.24, U4.24
Routing:
- net GND_MCU: track 760.0 -> 0.00 mm, vias 25 -> 0
- net 3.3V: track 569.6 -> 0.00 mm, vias 17 -> 0
- net VCC_5V: track 370.5 -> 0.00 mm, vias 4 -> 0
- net SCL_00: track 172.6 -> 0.00 mm, vias 3 -> 0
- net SDA_00: track 158.4 -> 0.00 mm, vias 5 -> 0
- net NEOPIXEL_02: track 127.2 -> 0.00 mm, vias 5 -> 0
- net NEOPIXEL_04: track 121.8 -> 0.00 mm, vias 3 -> 0
- net NEOPIXEL_01: track 112.4 -> 0.00 mm, vias 5 -> 0
- net VCC_5V_IN: track 83.6 -> 0.00 mm, vias 1 -> 0
- net NEOPIXEL_03: track 71.3 -> 0.00 mm, vias 3 -> 0
- net NEOPIXEL_08: track 60.4 -> 0.00 mm, vias 3 -> 0
- net 14_SX1: track 57.0 -> 0.00 mm, vias 2 -> 0
- net NEOPIXEL_06: track 56.2 -> 0.00 mm, vias 1 -> 0
- net 15_SX1: track 52.1 -> 0.00 mm, vias 2 -> 0
- net 7_SX1: track 51.2 -> 0.00 mm, vias 2 -> 0
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