File: Circuit/PCB/teensyMotors02_up_LED.brd (EAGLE design)
At the start: 72 x 150 mm, 65 parts, among them U1 SX1509

Commit message: board
Parts:
- removed U$5: SX1509, SX1509_s:SX1509
Connections:
- removed net N$10: U$5.2
- removed net N$11: U$5.3
- removed net N$15: U$5.4
- removed net N$16: U$5.5
- removed net N$7: U$5.0
- removed net N$8: U$5.1
Routing:
- net GND_MCU: track 792.0 -> 795.4 mm
- net 3.3V: track 247.4 -> 249.9 mm
- net VCC_5V: track 308.9 -> 311.2 mm
- net SDA_00: track 165.9 -> 167.2 mm
- net NEOPIXEL_03: track 36.9 -> 38.2 mm
- net MDIR_06: track 76.3 -> 77.6 mm
- net MSTEP_06: track 46.4 -> 47.6 mm
- net NEOPIXEL_05: track 44.5 -> 45.7 mm
- net NEOPIXEL_08: track 44.4 -> 45.7 mm
- net MSTEP_07: track 16.7 -> 17.9 mm
- net SCL_00: track 281.4 -> 282.6 mm
- net MSTEP_04: track 38.8 -> 40.0 mm
- net MDIR_05: track 18.1 -> 19.3 mm
- net MDIR_07: track 18.5 -> 19.8 mm
- net NEOPIXEL_02: track 51.6 -> 52.8 mm
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