File: Circuit/PCB/teensyMotors02_up_LED.sch (EAGLE design)
At the start: 65 parts, among them U1 SX1509

Commit message: circuit
Changed lines of the file:
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@@
 <text x="510.54" y="104.14" size="1.905" layer="97" rot="MR180">Allowable VCC1/2 Range:
 1.2-3.6V</text>
-<wire x1="408.94" y1="149.86" x2="561.34" y2="149.86" width="0.1524" layer="97"/>
-<wire x1="561.34" y1="-58.42" x2="561.34" y2="149.86" width="0.1524" layer="97"/>
-<wire x1="561.34" y1="-58.42" x2="358.14" y2="-58.42" width="0.1524" layer="97"/>
+<wire x1="408.94" y1="154.94" x2="736.6" y2="154.94" width="0.1524" layer="97"/>
+<wire x1="736.6" y1="-58.42" x2="736.6" y2="154.94" width="0.1524" layer="97"/>
+<wire x1="736.6" y1="-58.42" x2="358.14" y2="-58.42" width="0.1524" layer="97"/>
 <wire x1="358.14" y1="-58.42" x2="358.14" y2="142.24" width="0.1524" layer="97"/>
-<text x="358.14" y="147.32" size="6.4516" layer="97">IC2 MUX 01</text>
+<text x="358.14" y="152.4" size="6.4516" layer="97">IC2 MUX 01</text>
 </plain>
 <instances>
@@
 <instance part="JP3_TX7" gate="G$1" x="-40.64" y="121.92"/>
 <instance part="JP4_RX7" gate="G$1" x="-40.64" y="86.36"/>
-<instance part="U$5" gate="G$1" x="594.36" y="111.76"/>
+<instance part="U$5" gate="G$1" x="673.1" y="104.14"/>
 </instances>
 <busses>
@@
 <segment>
 <pinref part="U$5" gate="G$1" pin="0"/>
-<wire x1="586.74" y1="119.38" x2="576.58" y2="119.38" width="0.1524" layer="91"/>
+<wire x1="665.48" y1="111.76" x2="650.24" y2="111.76" width="0.1524" layer="91"/>
 </segment>
 </net>
@@
 <segment>
 <pinref part="U$5" gate="G$1" pin="1"/>
-<wire x1="586.74" y1="114.3" x2="576.58" y2="114.3" width="0.1524" layer="91"/>
+<wire x1="665.48" y1="106.68" x2="650.24" y2="106.68" width="0.1524" layer="91"/>
 </segment>
 </net>
@@
 <segment>
 <pinref part="U$5" gate="G$1" pin="2"/>
-<wire x1="586.74" y1="109.22" x2="579.12" y2="109.22" width="0.1524" layer="91"/>
+<wire x1="665.48" y1="101.6" x2="652.78" y2="101.6" width="0.1524" layer="91"/>
 </segment>
 </net>
@@
 <segment>
 <pinref part="U$5" gate="G$1" pin="3"/>
-<wire x1="586.74" y1="104.14" x2="576.58" y2="104.14" width="0.1524" layer="91"/>
+<wire x1="665.48" y1="96.52" x2="650.24" y2="96.52" width="0.1524" layer="91"/>
 </segment>
 </net>
@@
 <segment>
 <pinref part="U$5" gate="G$1" pin="4"/>
-<wire x1="586.74" y1="99.06" x2="576.58" y2="99.06" width="0.1524" layer="91"/>
+<wire x1="665.48" y1="91.44" x2="650.24" y2="91.44" width="0.1524" layer="91"/>
 </segment>
 </net>
@@
 <segment>
 <pinref part="U$5" gate="G$1" pin="5"/>
-<wire x1="586.74" y1="93.98" x2="574.04" y2="93.98" width="0.1524" layer="91"/>
-</segment>
-</net>
+<wire x1="665.48" y1="86.36" x2="647.7" y2="86.36" width="0.1524" layer="91"/>
+</segment>
+</net>

Commit message: board
Parts:
- removed U$5: SX1509, SX1509_s:SX1509
Connections:
- removed net N$10: U$5.2
- removed net N$11: U$5.3
- removed net N$15: U$5.4
- removed net N$16: U$5.5
- removed net N$7: U$5.0
- removed net N$8: U$5.1
Changed lines of the file:
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@@
 <part name="JP3_TX7" library="SparkFun-Jumpers" library_urn="urn:adsk.eagle:library:528" deviceset="JUMPER-SMT_3_1-NC_TRACE" device="_NO-SILK" package3d_urn="urn:adsk.eagle:package:39287/1"/>
 <part name="JP4_RX7" library="SparkFun-Jumpers" library_urn="urn:adsk.eagle:library:528" deviceset="JUMPER-SMT_3_1-NC_TRACE" device="_NO-SILK" package3d_urn="urn:adsk.eagle:package:39287/1"/>
-<part name="U$5" library="SX1509_s" deviceset="SX1509" device=""/>
 </parts>
 <sheets>
@@
 <text x="510.54" y="104.14" size="1.905" layer="97" rot="MR180">Allowable VCC1/2 Range:
 1.2-3.6V</text>
-<wire x1="408.94" y1="154.94" x2="736.6" y2="154.94" width="0.1524" layer="97"/>
-<wire x1="736.6" y1="-58.42" x2="736.6" y2="154.94" width="0.1524" layer="97"/>
-<wire x1="736.6" y1="-58.42" x2="358.14" y2="-58.42" width="0.1524" layer="97"/>
+<wire x1="408.94" y1="154.94" x2="576.58" y2="154.94" width="0.1524" layer="97"/>
+<wire x1="576.58" y1="-58.42" x2="576.58" y2="154.94" width="0.1524" layer="97"/>
+<wire x1="576.58" y1="-58.42" x2="358.14" y2="-58.42" width="0.1524" layer="97"/>
 <wire x1="358.14" y1="-58.42" x2="358.14" y2="142.24" width="0.1524" layer="97"/>
 <text x="358.14" y="152.4" size="6.4516" layer="97">IC2 MUX 01</text>
@@
 <instance part="JP3_TX7" gate="G$1" x="-40.64" y="121.92"/>
 <instance part="JP4_RX7" gate="G$1" x="-40.64" y="86.36"/>
-<instance part="U$5" gate="G$1" x="673.1" y="104.14"/>
 </instances>
 <busses>
@@
 </segment>
 </net>
-<net name="N$7" class="0">
-<segment>
-<pinref part="U$5" gate="G$1" pin="0"/>
-<wire x1="665.48" y1="111.76" x2="650.24" y2="111.76" width="0.1524" layer="91"/>
-</segment>
-</net>
-<net name="N$8" class="0">
-<segment>
-<pinref part="U$5" gate="G$1" pin="1"/>
-<wire x1="665.48" y1="106.68" x2="650.24" y2="106.68" width="0.1524" layer="91"/>
-</segment>
-</net>
-<net name="N$10" class="0">
-<segment>
-<pinref part="U$5" gate="G$1" pin="2"/>
-<wire x1="665.48" y1="101.6" x2="652.78" y2="101.6" width="0.1524" layer="91"/>
-</segment>
-</net>
-<net name="N$11" class="0">
-<segment>
-<pinref part="U$5" gate="G$1" pin="3"/>
-<wire x1="665.48" y1="96.52" x2="650.24" y2="96.52" width="0.1524" layer="91"/>
-</segment>
-</net>
-<net name="N$15" class="0">
-<segment>
-<pinref part="U$5" gate="G$1" pin="4"/>
-<wire x1="665.48" y1="91.44" x2="650.24" y2="91.44" width="0.1524" layer="91"/>
-</segment>
-</net>
-<net name="N$16" class="0">
-<segment>
-<pinref part="U$5" gate="G$1" pin="5"/>
-<wire x1="665.48" y1="86.36" x2="647.7" y2="86.36" width="0.1524" layer="91"/>
-</segment>
-</net>
