File: Circuit/PCB/LEDBox.brd (EAGLE design)
At the start: 28 x 28 mm, 12 parts, among them K1 D2F-5

Commit message: PCB
Parts:
- removed C3, C4: 0.1uf, microbuilder:1206
- removed K1: D2F-5, D2F-5:SHDR3W100P0X508_1X3_1280X580X5
- removed LED3, LED5: (no value), SK6812:LED5050
- added J3, J4, J5, J6: (no value), SparkFun-Connectors:1X02
- added R4: 10K, resistor:M0805
- added SWITCH_M1, SWITCH_M4: DTSM-3, switch-tact:DTSM-3
- C1, C2: device microbuilder:1206 -> rc-master-smd:C0805
- R1: value (none) -> 10K; device eagle-ltspice:R3216 -> resistor:M0805
- moved C2 21.1 mm to (17.9, 26.1), flipped to the bottom, turned to 180 degrees
- moved LED2 19.3 mm to (4.93, 5.63)
- moved J1 13.9 mm to (19.9, 9.47), turned to 90 degrees
- moved R1 10.9 mm to (8.89, 25.9), flipped to the bottom, turned to 180 degrees
- moved LED1 2.96 mm to (22.5, 22.7)
- moved C1 2.14 mm to (17.9, 23.2), flipped to the bottom, turned to 180 degrees
- moved J2 2.14 mm to (25.0, 13.5), flipped to the bottom, turned to 270 degrees
Connections:
- net LDIN renamed NEO_IN
- net SCL renamed DIO_IN
- removed net N$3: LED3.2-DOUT, LED5.4-DIN
- removed net N$6: K1.3
- removed net SDA: J1.2, J2.5
- removed net SDIN: J2.4, K1.2, R1.2
- new net SWD_IN: J2.4, R4.2, SWITCH_M4.2
- new net SWU_IN: J1.2, J2.5, R1.2, SWITCH_M1.2
- net GND: now also C1.1, C2.1, R4.1; no longer C1.2, C2.2, C3.2, C4.2, LED3.3-GND, LED5.3-GND
- net N$2: no longer LED3.4-DIN
- net VCC: now also C1.2, C2.2, SWITCH_M1.1, SWITCH_M4.1; no longer C1.1, C2.1, C3.1, C4.1, K1.1, LED3.1-VDD, LED5.1-VDD
Routing:
- net SWU_IN: track 0.00 -> 41.3 mm
- net VCC: track 86.7 -> 50.6 mm
- net GND: track 35.1 -> 0.00 mm, vias 4 -> 0
- net SDIN: track 32.2 -> 0.00 mm
- net N$2: track 26.7 -> 0.00 mm, vias 2 -> 0
- net SWD_IN: track 0.00 -> 26.6 mm, vias 0 -> 2
- net N$3: track 20.1 -> 0.00 mm
- net NEO_IN: track 10.6 -> 29.5 mm, vias 0 -> 1
- net SDA: track 14.9 -> 0.00 mm, vias 1 -> 0
- net N$1: track 26.4 -> 39.0 mm, vias 2 -> 0
- net DIO_IN: track 15.2 -> 4.56 mm, vias 1 -> 0
Other:
- outline, holes or cut-outs redrawn
- board text added: "1"
- board text added: "2"
- board text added: "down"
- board text removed: "SCL"
- board text removed: "SDA"

Commit message: circuit update
Parts:
- moved SWITCH_M4 2.59 mm to (14.5, 24.7)
- moved SWITCH_M1 0.92 mm to (14.5, 3.30)
Connections:
- net GND: now also SWITCH_M1.1, SWITCH_M4.1; no longer R1.1, R4.1
- net VCC: now also R1.1, R4.1; no longer SWITCH_M1.1, SWITCH_M4.1
Routing:
- net VCC: track 50.6 -> 0.00 mm
- net SWU_IN: track 41.3 -> 0.00 mm
- net N$1: track 39.0 -> 0.00 mm
- net NEO_IN: track 29.5 -> 0.00 mm, vias 1 -> 0
- net SWD_IN: track 26.6 -> 0.00 mm, vias 2 -> 0
- net DIO_IN: track 4.56 -> 0.00 mm

Commit message: board
Parts:
- removed J3, J4, J5, J6: (no value), SparkFun-Connectors:1X02
- removed R1, R4: 10K, resistor:M0805
- added C3, C4: 0.1uf, rc-master-smd:C0805
- added JP1: JUMPER-SMT_2_NO_NO-SILK_ROUND, SparkFun-Jumpers:SMT-JUMPER_2_NO_NO-SILK_ROUND
- added LED3, LED4: (no value), SK6812:LED5050_W
- added R13_S, R1_UP, R4_DOWN: 10K, resistor:M0805
- added SW6: B3F-1000, Switch:B3F-1000
- LED1, LED2: device SK6812:LED5050 -> SK6812:LED5050_W
- moved C2 13.7 mm to (7.73, 16.9), flipped to the top
- moved C1 10.9 mm to (7.73, 19.4), flipped to the top
- moved LED1 1.70 mm to (23.2, 24.2)
- moved LED2 1.27 mm to (4.93, 4.36)
- moved SWITCH_M1 1.14 mm to (14.0, 4.32)
- moved SWITCH_M4 0.80 mm to (14.2, 24.0)
- moved J1 0.57 mm to (19.6, 9.98)
Connections:
- new net N$4: JP1.2, LED3.4-DIN
- new net N$5: LED4.2-DOUT
- new net N$6: LED3.2-DOUT, LED4.4-DIN
- net GND: now also C3.1, C4.1, LED3.3-GND, LED4.3-GND, R13_S.1, R1_UP.1, R4_DOWN.1; no longer SWITCH_M1.1, SWITCH_M4.1
- net N$2: now also JP1.1
- net SWD_IN: now also R4_DOWN.2; no longer R4.2
- net SWU_IN: now also R13_S.2, R1_UP.2, SW6.3; no longer R1.2
- net VCC: now also C3.2, C4.2, LED3.1-VDD, LED4.1-VDD, SW6.1, SWITCH_M1.1, SWITCH_M4.1; no longer R1.1, R4.1
Routing:
- net VCC: track 0.00 -> 109.7 mm, vias 0 -> 3
- net GND: track 0.00 -> 92.4 mm, vias 0 -> 8
- net SWU_IN: track 0.00 -> 71.6 mm, vias 0 -> 2
- net N$6: track 0.00 -> 53.7 mm, vias 0 -> 2
- net N$1: track 0.00 -> 42.9 mm, vias 0 -> 2
- net SWD_IN: track 0.00 -> 37.4 mm, vias 0 -> 2
- net N$2: track 0.00 -> 14.2 mm, vias 0 -> 3
- net NEO_IN: track 0.00 -> 11.7 mm, vias 0 -> 1
- net N$4: track 0.00 -> 10.3 mm, vias 0 -> 3
- net DIO_IN: track 0.00 -> 4.51 mm
Other:
- board text added: "3"
- board text added: "4"
- board text added: "DIO"
- board text added: "NEO"
- board text added: "SWD"
- board text added: "SWU"
- board text added: "UP"

Commit message: merge
Parts:
- added R13_S1: 10K, resistor:M0805
- added SWD: B3F-1000, Switch:B3F-1000
- moved C4 15.8 mm to (23.1, 7.62), turned to 0 degrees
- moved C1 15.6 mm to (23.3, 20.3), turned to 0 degrees
- moved C2 9.56 mm to (4.93, 7.78), turned to 0 degrees
- moved C3 9.25 mm to (4.83, 20.3), turned to 0 degrees
- moved R4_DOWN 5.04 mm to (7.11, 17.0)
- moved R1_UP 2.34 mm to (2.79, 17.0)
- moved LED2 0.76 mm to (4.93, 3.60)
- moved SWITCH_M4 0.51 mm to (14.7, 24.0)
- moved LED4 0.51 mm to (23.1, 3.56)
- renumbered SW6 to SWU
Connections:
- net GND: now also R13_S1.1
- net SWD_IN: now also R13_S1.2, SWD.3
- net VCC: now also SWD.1
Routing:
- net SWU_IN: track 71.6 -> 45.1 mm, vias 2 -> 1
- net N$6: track 53.7 -> 33.2 mm
- net NEO_IN: track 11.7 -> 28.5 mm
- net GND: track 92.4 -> 78.8 mm, vias 8 -> 9
- net VCC: track 109.7 -> 116.7 mm, vias 3 -> 4
- net N$2: track 14.2 -> 7.56 mm, vias 3 -> 1
- net SWD_IN: track 37.4 -> 34.3 mm, vias 2 -> 1
- net N$1: track 42.9 -> 43.5 mm
- net N$4: track 10.3 -> 10.2 mm, vias 3 -> 1
