File: Circuit/PCB/LEDBox.sch (EAGLE design)
At the start: 12 parts, among them K1 D2F-5

Commit message: PCB
Parts:
- removed C3, C4: 0.1uf, microbuilder:CAP_CERAMIC1206
- removed K1: D2F-5, D2F-5:D2F-5
- removed LED3, LED5: (no value), SK6812:SK6812_5050
- added J3, J4, J5, J6: (no value), SparkFun-Connectors:CONN_02
- added R4: 10K, resistor:R-US_M0805
- added SWITCH_M1, SWITCH_M4: DTSM-3, switch-tact:DTSM-3
- C1, C2: device microbuilder:CAP_CERAMIC1206 -> rc-master-smd:C_0805
- R1: value (none) -> 10K; device eagle-ltspice:RR3216 -> resistor:R-US_M0805
Connections:
- net LDIN renamed NEO_IN
- net SCL renamed DIO_IN
- removed net N$3: LED3.DO, LED5.DI
- removed net N$6: K1.NC
- removed net SDA: J1.2, J2.5
- removed net SDIN: J2.4, K1.NO, R1.2
- new net SWD_IN: J2.4, R4.2, SWITCH_M4.2
- new net SWU_IN: J1.2, J2.5, R1.2, SWITCH_M1.2
- net GND: now also C1.1, C2.1, R4.1; no longer C1.P$2, C2.P$2, C3.P$2, C4.P$2, LED3.GND, LED5.GND
- net N$2: no longer LED3.DI
- net VCC: now also C1.2, C2.2, SWITCH_M1.1, SWITCH_M4.1; no longer C1.P$1, C2.P$1, C3.P$1, C4.P$1, K1.COM, LED3.VDD, LED5.VDD
Other:
- moved on the sheet: C1, C2, J1, J2, LED1, LED2

Commit message: circuit update
Connections:
- net GND: now also SWITCH_M1.1, SWITCH_M4.1; no longer R1.1, R4.1
- net VCC: now also R1.1, R4.1; no longer SWITCH_M1.1, SWITCH_M4.1
Changed lines of the file:
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@@
-</segment>
-<segment>
-<pinref part="R4" gate="G$1" pin="1"/>
-<wire x1="109.22" y1="5.08" x2="109.22" y2="2.54" width="0.1524" layer="91"/>
-<label x="109.22" y="2.54" size="1.016" layer="95" rot="R270" xref="yes"/>
 </segment>
 <segment>
@@
 </segment>
 <segment>
-<pinref part="R1" gate="G$1" pin="1"/>
-<wire x1="71.12" y1="-20.32" x2="71.12" y2="-22.86" width="0.1524" layer="91"/>
-<label x="71.12" y="-22.86" size="1.016" layer="95" rot="R270" xref="yes"/>
+<pinref part="SWITCH_M4" gate="G$1" pin="1"/>
+<wire x1="88.9" y1="17.78" x2="78.74" y2="17.78" width="0.1524" layer="91"/>
+<label x="76.2" y="17.78" size="1.016" layer="95" rot="R180" xref="yes"/>
+</segment>
+<segment>
+<pinref part="SWITCH_M1" gate="G$1" pin="1"/>
+<wire x1="50.8" y1="-7.62" x2="40.64" y2="-7.62" width="0.1524" layer="91"/>
+<label x="38.1" y="-7.62" size="1.016" layer="95" rot="R180" xref="yes"/>
 </segment>
 </net>
@@
 <wire x1="10.16" y1="38.1" x2="17.78" y2="38.1" width="0.1524" layer="91"/>
 <label x="17.78" y="38.1" size="1.016" layer="95" xref="yes"/>
-</segment>
-<segment>
-<pinref part="SWITCH_M4" gate="G$1" pin="1"/>
-<wire x1="88.9" y1="17.78" x2="78.74" y2="17.78" width="0.1524" layer="91"/>
-<label x="76.2" y="17.78" size="1.016" layer="95" rot="R180" xref="yes"/>
 </segment>
 <segment>
@@
 </segment>
 <segment>
-<pinref part="SWITCH_M1" gate="G$1" pin="1"/>
-<wire x1="50.8" y1="-7.62" x2="40.64" y2="-7.62" width="0.1524" layer="91"/>
-<label x="38.1" y="-7.62" size="1.016" layer="95" rot="R180" xref="yes"/>
+<pinref part="R4" gate="G$1" pin="1"/>
+<wire x1="109.22" y1="5.08" x2="109.22" y2="2.54" width="0.1524" layer="91"/>
+<label x="109.22" y="2.54" size="1.016" layer="95" rot="R270" xref="yes"/>
+</segment>
+<segment>
+<pinref part="R1" gate="G$1" pin="1"/>
+<wire x1="71.12" y1="-20.32" x2="71.12" y2="-22.86" width="0.1524" layer="91"/>
+<label x="71.12" y="-22.86" size="1.016" layer="95" rot="R270" xref="yes"/>
 </segment>
 </net>

Commit message: board
Parts:
- removed J3, J4, J5, J6: (no value), SparkFun-Connectors:CONN_02
- removed R1, R4: 10K, resistor:R-US_M0805
- added C3, C4: 0.1uf, rc-master-smd:C_0805
- added JP1: JUMPER-SMT_2_NO_NO-SILK_ROUND, SparkFun-Jumpers:JUMPER-SMT_2_NO_NO-SILK_ROUND
- added LED3, LED4: (no value), SK6812:SK6812_5050W
- added R13_S, R1_UP, R4_DOWN: 10K, resistor:R-US_M0805
- added SW6: B3F-1000, Switch:B3F-1000
- LED1, LED2: device SK6812:SK6812_5050 -> SK6812:SK6812_5050W
Connections:
- new net N$4: JP1.2, LED3.DI
- new net N$5: LED4.DO
- new net N$6: LED3.DO, LED4.DI
- net GND: now also C3.1, C4.1, LED3.GND, LED4.GND, R13_S.1, R1_UP.1, R4_DOWN.1; no longer SWITCH_M1.1, SWITCH_M4.1
- net N$2: now also JP1.1
- net SWD_IN: now also R4_DOWN.2; no longer R4.2
- net SWU_IN: now also R13_S.2, R1_UP.2, SW6.3; no longer R1.2
- net VCC: now also C3.2, C4.2, LED3.VDD, LED4.VDD, SW6.1, SWITCH_M1.1, SWITCH_M4.1; no longer R1.1, R4.1
Other:
- moved on the sheet: J1, J2, SWITCH_M1, SWITCH_M4

Commit message: merge
Parts:
- added R13_S1: 10K, resistor:R-US_M0805
- added SWD: B3F-1000, Switch:B3F-1000
- renumbered SW6 to SWU
Connections:
- net GND: now also R13_S1.1
- net SWD_IN: now also R13_S1.2, SWD.3
- net VCC: now also SWD.1
Changed lines of the file:
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@@
 <part name="LED4" library="SK6812" deviceset="SK6812" device="_5050W"/>
 <part name="C4" library="rc-master-smd" deviceset="C_" device="0805" value="0.1uf"/>
-<part name="SW6" library="Switch" library_urn="urn:adsk.eagle:library:11396471" deviceset="B3F-1000" device="" package3d_urn="urn:adsk.eagle:package:10899221/2"/>
+<part name="SWU" library="Switch" library_urn="urn:adsk.eagle:library:11396471" deviceset="B3F-1000" device="" package3d_urn="urn:adsk.eagle:package:10899221/2"/>
 <part name="R13_S" library="resistor" library_urn="urn:adsk.eagle:library:348" deviceset="R-US_" device="M0805" package3d_urn="urn:adsk.eagle:package:26079/1" value="10K"/>
 <part name="JP1" library="SparkFun-Jumpers" library_urn="urn:adsk.eagle:library:528" deviceset="JUMPER-SMT_2_NO" device="_NO-SILK_ROUND" package3d_urn="urn:adsk.eagle:package:39278/1"/>
+<part name="SWD" library="Switch" library_urn="urn:adsk.eagle:library:11396471" deviceset="B3F-1000" device="" package3d_urn="urn:adsk.eagle:package:10899221/2"/>
+<part name="R13_S1" library="resistor" library_urn="urn:adsk.eagle:library:348" deviceset="R-US_" device="M0805" package3d_urn="urn:adsk.eagle:package:26079/1" value="10K"/>
 </parts>
 <sheets>
@@
 <instance part="LED4" gate="G$1" x="269.24" y="76.2"/>
 <instance part="C4" gate="G$1" x="287.02" y="93.98" rot="R90"/>
-<instance part="SW6" gate="G$1" x="213.36" y="7.62"/>
+<instance part="SWU" gate="G$1" x="213.36" y="7.62"/>
 <instance part="R13_S" gate="G$1" x="238.76" y="0" rot="R90"/>
 <instance part="JP1" gate="G$1" x="157.48" y="73.66"/>
+<instance part="SWD" gate="G$1" x="218.44" y="-33.02"/>
+<instance part="R13_S1" gate="G$1" x="243.84" y="-40.64" rot="R90"/>
 </instances>
 <busses>
@@
 <label x="238.76" y="-10.16" size="1.016" layer="95" rot="R270" xref="yes"/>
 </segment>
+<segment>
+<pinref part="R13_S1" gate="G$1" pin="1"/>
+<wire x1="243.84" y1="-45.72" x2="243.84" y2="-50.8" width="0.1524" layer="91"/>
+<label x="243.84" y="-50.8" size="1.016" layer="95" rot="R270" xref="yes"/>
+</segment>
 </net>
 <net name="VCC" class="0">
@@
 </segment>
 <segment>
-<pinref part="SW6" gate="G$1" pin="1"/>
+<pinref part="SWU" gate="G$1" pin="1"/>
 <wire x1="223.52" y1="2.54" x2="228.6" y2="2.54" width="0.1524" layer="91"/>
 <wire x1="228.6" y1="2.54" x2="228.6" y2="-7.62" width="0.1524" layer="91"/>
 <label x="228.6" y="-10.16" size="1.016" layer="95" rot="R270" xref="yes"/>
+</segment>
+<segment>
+<pinref part="SWD" gate="G$1" pin="1"/>
+<wire x1="228.6" y1="-38.1" x2="233.68" y2="-38.1" width="0.1524" layer="91"/>
+<wire x1="233.68" y1="-38.1" x2="233.68" y2="-48.26" width="0.1524" layer="91"/>
+<label x="233.68" y="-50.8" size="1.016" layer="95" rot="R270" xref="yes"/>
 </segment>
 </net>
@@
 <label x="154.94" y="20.32" size="1.016" layer="95" xref="yes"/>
 </segment>
+<segment>
+<pinref part="SWD" gate="G$1" pin="3"/>
+<wire x1="228.6" y1="-30.48" x2="243.84" y2="-30.48" width="0.1524" layer="91"/>
+<pinref part="R13_S1" gate="G$1" pin="2"/>
+<wire x1="243.84" y1="-30.48" x2="264.16" y2="-30.48" width="0.1524" layer="91"/>
+<wire x1="243.84" y1="-35.56" x2="243.84" y2="-30.48" width="0.1524" layer="91"/>
+<junction x="243.84" y="-30.48"/>
+<label x="264.16" y="-30.48" size="1.016" layer="95" xref="yes"/>
+</segment>
 </net>
 <net name="SWU_IN" class="0">
@@
 </segment>
 <segment>
-<pinref part="SW6" gate="G$1" pin="3"/>
+<pinref part="SWU" gate="G$1" pin="3"/>
 <wire x1="223.52" y1="10.16" x2="238.76" y2="10.16" width="0.1524" layer="91"/>
 <pinref part="R13_S" gate="G$1" pin="2"/>
