File: Circuit/PCB/teensyMotors02_up_LED_SX.brd (EAGLE design)
At the start: 72 x 150 mm, 59 parts

Commit message: circuit
Parts:
- removed C15: 100uF, SparkFun-Capacitors:PANASONIC_D
- removed C9: 2.2uf, SparkFun-Capacitors:0603-CAP
- removed D1, D2: S2M, s2x_10:DO214AA
- removed U$2: (no value), 1zac:VSSOP(8)
- added C1: 1.5uf, SparkFun-Capacitors:0603-CAP
- added R1: 1K, SparkFun-Resistors:0603-RES
- added SMAJ24A, SMAT70A, Z3120V: S2M, s2x_10:DO214AA
- added U1: LTC4359CMS8PBF, LTC4359CMS8PBF:MSOP-8_MS
- moved C10 17.5 mm to (29.0, 61.0), turned to 90 degrees
- moved C4 9.41 mm to (62.5, 85.9), turned to 270 degrees
- moved C7 7.12 mm to (18.3, 74.9)
- moved C8 6.19 mm to (15.5, 74.9)
- moved CAN_INPUT1 6.05 mm to (69.8, 68.9)
- moved CAN_INPUT5 5.33 mm to (22.6, 8.38)
- moved J1 5.00 mm to (67.1, 80.0), turned to 180 degrees
- moved C6 4.34 mm to (65.3, 85.9), turned to 90 degrees
- moved U$1 4.32 mm to (54.4, 86.1)
- moved R10 3.31 mm to (69.1, 55.4)
- moved D3 3.18 mm to (56.4, 70.4)
- moved U$4 2.87 mm to (7.46, 90.1)
- moved R8 2.34 mm to (67.8, 85.9), turned to 270 degrees
- moved CAN_INPUT 2.09 mm to (6.63, 68.9)
- moved STATUS_LED 2.05 mm to (69.1, 60.2)
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Connections:
- removed net N$5: C9.2, U$2.VCAPL
- net GND_MCU: now also R1.2; no longer C15.-, D2.C
- net N$12: now also SMAJ24A.A, SMAT70A.A; no longer D1.A, D2.A
- net N$2: now also U$4.1, U1.1, Z3120V.C; no longer C9.1, U$2.VCAPH
- net N$4: now also C1.2, R1.1, SMAJ24A.C, U1.6; no longer U$2.GDRIVE, U$2.GPD, U$4.1
- net REG_5V: now also C1.1, U1.8; no longer C15.+, U$2.CATHODE
- net VCC_MCU: now also SMAT70A.C, U1.2, U1.4, U1.5, Z3120V.A; no longer D1.C, U$2.ANODE
Routing:
- net GND_MCU: track 0.00 -> 603.9 mm, vias 0 -> 55
- net VCC_M: track 0.00 -> 408.8 mm
- net VCC_5V: track 0.00 -> 401.2 mm, vias 0 -> 15
- net MMS1: track 0.00 -> 312.0 mm, vias 0 -> 11
- net SCL_00: track 0.00 -> 290.2 mm, vias 0 -> 21
- net 3.3V: track 0.00 -> 286.7 mm, vias 0 -> 14
- net TRQ1: track 0.00 -> 279.5 mm, vias 0 -> 18
- net SDA_00: track 0.00 -> 274.3 mm, vias 0 -> 13
- net MMS2: track 0.00 -> 273.8 mm, vias 0 -> 15
- net TRQ2: track 0.00 -> 265.5 mm, vias 0 -> 12
- net 13_SX0: track 0.00 -> 144.6 mm, vias 0 -> 5
- net MDIR_01: track 0.00 -> 137.9 mm, vias 0 -> 3
- net 14_SX0: track 0.00 -> 127.0 mm, vias 0 -> 7
- net 10_SX0: track 0.00 -> 118.7 mm, vias 0 -> 7
- net STATUS_PIN: track 0.00 -> 116.7 mm, vias 0 -> 10
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
Commit message: board
Connections:
- net REG_5V: now also S1.3; no longer S1.6
Routing:
- net TRQ1: track 279.5 -> 0.00 mm, vias 18 -> 0
- net REG_5V: track 71.2 -> 78.0 mm, vias 2 -> 4

Commit message: board
Parts:
- I2C, NOE_PIXELS: value TMMH-105-12 -> (none); device TMMH-105-XX-XX-DV:TMMH-105-12 -> SparkFun-Connectors:2X6_SMD
- R4, R8: value 60 -> 120Ohms
- U$3: value TEENSY_4.0_WITH_SMD_HEADER_PINSTEENSY_4.0_SMD -> TEENSY_4.0_WITH_SMD_HEADER_PINS; device Teensy4:TEENSY_4.0_SMD -> Teensy4:TEENSY_4.0_WITH_SMD_HEADER_PINS
- moved MC8 19.1 mm to (68.9, 100.3)
- moved CM_08 13.7 mm to (26.4, 101.6), turned to 90 degrees
- moved CM_07 11.9 mm to (38.0, 145.5)
- moved CM_03 11.2 mm to (38.5, 13.0)
- moved MOTOR_08 10.7 mm to (42.7, 102.6), turned to 0 degrees
- moved U$3 9.14 mm to (38.2, 100.3)
- moved CAN_INPUT4 4.07 mm to (54.4, 8.64)
- moved MOTOR_07 4.06 mm to (38.1, 126.6)
- moved MC6 2.34 mm to (27.8, 141.8)
- moved MOTOR_05 2.18 mm to (61.9, 117.8)
- moved CM_05 1.93 mm to (62.0, 130.0)
- moved MC7 1.61 mm to (48.2, 141.6)
- moved MC5 1.55 mm to (68.9, 141.6)
- moved MOTOR_06 1.52 mm to (14.1, 117.5)
- moved CAN_INPUT5 1.27 mm to (21.3, 8.38)
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Routing:
- net TRQ1: track 0.00 -> 296.1 mm, vias 0 -> 15
- net CAN_H: track 86.8 -> 262.2 mm, vias 2 -> 14
- net GND_MCU: track 603.9 -> 706.3 mm, vias 55 -> 61
- net NEOPIXEL_04: track 53.6 -> 134.3 mm, vias 2 -> 7
- net SDA_00: track 274.3 -> 346.8 mm, vias 13 -> 12
- net 13_SX0: track 144.6 -> 214.8 mm, vias 5 -> 11
- net MDIR_01: track 137.9 -> 204.9 mm, vias 3 -> 5
- net VCC_5V: track 401.2 -> 459.5 mm, vias 15 -> 26
- net MSTEP_06: track 44.0 -> 102.1 mm
- net VCC_M: track 408.8 -> 463.0 mm
- net 12_SX0: track 86.5 -> 136.5 mm, vias 7 -> 9
- net 15_SX0: track 50.2 -> 97.9 mm, vias 7 -> 9
- net MSTEP_08: track 59.7 -> 13.9 mm, vias 3 -> 1
- net 14_SX0: track 127.0 -> 172.7 mm
- net CAN_RX2: track 107.2 -> 152.2 mm, vias 8 -> 7
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Other:
- board text added: "-"
- board text removed: "ADDR"
- board text removed: "ADDR0"

Commit message: merge
Parts:
- removed U$4: (no value), v-reg-2:TO263-3
- added D1: BSC010NE2LSI, BSC010NE2LSI:SOFL127P515X615X110-9N
Connections:
- net N$2: now also D1.4; no longer U$4.1
- net REG_5V: now also D1.5, D1.6, D1.7, D1.8, D1.9; no longer U$4.4
- net VCC_MCU: now also D1.1, D1.2, D1.3; no longer U$4.3
Routing:
- net NEOPIXEL_04: track 134.3 -> 99.1 mm, vias 7 -> 6
- net SCL_00: track 260.7 -> 239.1 mm, vias 9 -> 12
- net MSTEP_05: track 33.7 -> 29.1 mm, vias 1 -> 2
- net GND_MCU: track 706.3 -> 710.2 mm, vias 61 -> 66
- net VCC_MCU: track 47.0 -> 50.1 mm
- net N$2: track 25.9 -> 23.3 mm
- net REG_5V: track 78.2 -> 80.5 mm, vias 4 -> 7
- net MMS2: track 297.6 -> 299.9 mm
- net SDA_00: track 346.8 -> 345.2 mm
- net MMS1: track 315.5 -> 314.3 mm
- net CAN_H: track 262.2 -> 262.8 mm
- net CAN_RX3: track 19.0 -> 18.9 mm, vias 0 -> 2
