File: Circuit/PCB/teensyMotors02_up_LED_SX.sch (EAGLE design)
At the start: 59 parts

Commit message: circuit
Parts:
- removed C15: 100uF, SparkFun-Capacitors:100UF-POLAR-25V-20%(ELEC)
- removed C9: 2.2uf, SparkFun-Capacitors:0.1UF-25V(+80/-20%)(0603)
- removed D1, D2: S2M, s2x_10:S2M
- removed U$2: (no value), 1zac:LM74610-Q1
- added C1: 1.5uf, SparkFun-Capacitors:0.1UF-25V(+80/-20%)(0603)
- added R1: 1K, SparkFun-Resistors:10KOHM-1/10W-1%(0603)0603
- added SMAJ24A, SMAT70A, Z3120V: S2M, s2x_10:S2M
- added U1: LTC4359CMS8PBF, LTC4359CMS8PBF:LTC4359CMS8PBF
Connections:
- removed net N$5: C9.2, U$2.VCAPL
- net GND_MCU: now also R1.2; no longer C15.-, D2.C
- net N$12: now also SMAJ24A.A, SMAT70A.A; no longer D1.A, D2.A
- net N$2: now also U$4.IN, U1.GATE, Z3120V.C; no longer C9.1, U$2.VCAPH
- net N$4: now also C1.2, R1.1, SMAJ24A.C, U1.VSS; no longer U$2.GDRIVE, U$2.GPD, U$4.IN
- net REG_5V: now also C1.1, U1.OUT; no longer C15.+, U$2.CATHODE
- net VCC_MCU: now also SMAT70A.C, U1.*SHDN, U1.IN, U1.SOURCE, Z3120V.A; no longer D1.C, U$2.ANODE
Other:
- moved on the sheet: C7, C8, POWER_M, POWER_MCU, S1, U$4

Commit message: board
Connections:
- net REG_5V: now also S1.3; no longer S1.6
Changed lines of the file:
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@@
 </segment>
 <segment>
-<pinref part="S1" gate="G$1" pin="6"/>
-<wire x1="-22.86" y1="22.86" x2="-17.78" y2="22.86" width="0.1524" layer="91"/>
-<label x="-17.78" y="22.86" size="1.016" layer="95" xref="yes"/>
+<pinref part="S1" gate="G$1" pin="3"/>
+<wire x1="-22.86" y1="30.48" x2="-17.78" y2="30.48" width="0.1524" layer="91"/>
+<label x="-17.78" y="30.48" size="1.016" layer="95" xref="yes"/>
 </segment>
 </net>

Commit message: board
Parts:
- I2C, NOE_PIXELS: value TMMH-105-12 -> (none); device TMMH-105-XX-XX-DV:TMMH-105-12 -> SparkFun-Connectors:CONN_06X2SMD_FEMALE
- R4, R8: value 60 -> 120Ohms
- U$3: value TEENSY_4.0_WITH_SMD_HEADER_PINSTEENSY_4.0_SMD -> TEENSY_4.0_WITH_SMD_HEADER_PINS; device Teensy4:TEENSY_4.0_WITH_SMD_HEADER_PINSTEENSY_4.0_SMD -> Teensy4:TEENSY_4.0_WITH_SMD_HEADER_PINS
Other:
- moved on the sheet: I2C, NOE_PIXELS

Commit message: merge
Parts:
- removed U$4: (no value), v-reg-2:BUK
- added D1: BSC010NE2LSI, BSC010NE2LSI:BSC010NE2LSI
Connections:
- net N$2: now also D1.G; no longer U$4.IN
- net REG_5V: now also D1.D; no longer U$4.GND
- net VCC_MCU: now also D1.S; no longer U$4.OUT
Changed lines of the file:
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@@
 <part name="SMAT70A" library="s2x_10" deviceset="S2*" device="" technology="M"/>
 <part name="SMAJ24A" library="s2x_10" deviceset="S2*" device="" technology="M"/>
-<part name="U$4" library="v-reg-2" deviceset="BUK" device=""/>
 <part name="S1" library="SparkFun-Switches" library_urn="urn:adsk.eagle:library:535" deviceset="SWITCH-DPDT" device="-SMD-AYZ0202" package3d_urn="urn:adsk.eagle:package:40160/1">
 <attribute name="SPICEPREFIX" value="X"/>
@@
 <part name="C1" library="SparkFun-Capacitors" deviceset="0.1UF-25V(+80/-20%)(0603)" device="" value="1.5uf"/>
 <part name="R1" library="SparkFun-Resistors" library_urn="urn:adsk.eagle:library:532" deviceset="10KOHM-1/10W-1%(0603)" device="0603" value="1K"/>
+<part name="D1" library="BSC010NE2LSI" deviceset="BSC010NE2LSI" device=""/>
 </parts>
 <sheets>
@@
 <instance part="SMAT70A" gate="G$1" x="-154.94" y="12.7" rot="R90"/>
 <instance part="SMAJ24A" gate="G$1" x="-154.94" y="0" rot="R270"/>
-<instance part="U$4" gate="G$1" x="-86.36" y="22.86" rot="R90"/>
 <instance part="S1" gate="G$1" x="-27.94" y="30.48" smashed="yes">
 <attribute name="NAME" x="-27.94" y="38.354" size="1.778" layer="95" font="vector" align="bottom-center"/>
@@
 <attribute name="VALUE" x="-120.65" y="-54.102" size="1.778" layer="96"/>
 </instance>
+<instance part="D1" gate="G$1" x="-83.82" y="22.86" rot="R270"/>
 </instances>
 <busses>
@@
 <wire x1="-73.66" y1="-25.4" x2="-71.12" y2="-25.4" width="0.1524" layer="91"/>
 <wire x1="-71.12" y1="-25.4" x2="-71.12" y2="-38.1" width="0.1524" layer="91"/>
-<pinref part="U$4" gate="G$1" pin="OUT"/>
 <pinref part="SMAT70A" gate="G$1" pin="C"/>
 <wire x1="-180.34" y1="30.48" x2="-180.34" y2="-12.7" width="0.1524" layer="91"/>
@@
 <wire x1="-154.94" y1="30.48" x2="-147.32" y2="30.48" width="0.1524" layer="91"/>
 <label x="-180.34" y="-12.7" size="1.016" layer="95" rot="R270" xref="yes"/>
-<wire x1="-147.32" y1="30.48" x2="-86.36" y2="30.48" width="0.1524" layer="91"/>
 <wire x1="-147.32" y1="2.54" x2="-147.32" y2="30.48" width="0.1524" layer="91"/>
 <junction x="-147.32" y="2.54"/>
+<pinref part="D1" gate="G$1" pin="S"/>
+<wire x1="-91.44" y1="22.86" x2="-137.16" y2="22.86" width="0.1524" layer="91"/>
+<wire x1="-137.16" y1="22.86" x2="-139.7" y2="22.86" width="0.1524" layer="91"/>
+<wire x1="-139.7" y1="22.86" x2="-139.7" y2="30.48" width="0.1524" layer="91"/>
+<wire x1="-139.7" y1="30.48" x2="-147.32" y2="30.48" width="0.1524" layer="91"/>
 <junction x="-147.32" y="30.48"/>
 </segment>
@@
 <junction x="-53.34" y="22.86"/>
 <wire x1="-53.34" y1="22.86" x2="-66.04" y2="22.86" width="0.1524" layer="91"/>
-<pinref part="U$4" gate="G$1" pin="GND"/>
 <label x="-53.34" y="35.56" size="1.016" layer="95" rot="R90" xref="yes"/>
 <pinref part="U1" gate="A" pin="OUT"/>
-<wire x1="-66.04" y1="22.86" x2="-78.74" y2="22.86" width="0.1524" layer="91"/>
 <wire x1="-73.66" y1="-17.78" x2="-66.04" y2="-17.78" width="0.1524" layer="91"/>
 <wire x1="-66.04" y1="-17.78" x2="-66.04" y2="22.86" width="0.1524" layer="91"/>
+<pinref part="C1" gate="G$1" pin="1"/>
+<pinref part="D1" gate="G$1" pin="D"/>
+<wire x1="-76.2" y1="22.86" x2="-66.04" y2="22.86" width="0.1524" layer="91"/>
 <junction x="-66.04" y="22.86"/>
-<pinref part="C1" gate="G$1" pin="1"/>
 </segment>
 <segment>
@@
 <net name="N$2" class="0">
 <segment>
-<pinref part="U$4" gate="G$1" pin="IN"/>
-<wire x1="-86.36" y1="15.24" x2="-86.36" y2="2.54" width="0.1524" layer="91"/>
 <wire x1="-86.36" y1="2.54" x2="-86.36" y2="-7.62" width="0.1524" layer="91"/>
 <wire x1="-86.36" y1="-7.62" x2="-142.24" y2="-7.62" width="0.1524" layer="91"/>
 <pinref part="Z3120V" gate="G$1" pin="C"/>
 <wire x1="-111.76" y1="2.54" x2="-86.36" y2="2.54" width="0.1524" layer="91"/>
-<junction x="-86.36" y="2.54"/>
 <pinref part="U1" gate="A" pin="GATE"/>
 <wire x1="-139.7" y1="-17.78" x2="-142.24" y2="-17.78" width="0.1524" layer="91"/>
 <wire x1="-142.24" y1="-17.78" x2="-142.24" y2="-7.62" width="0.1524" layer="91"/>
-</segment>
-</net>
+<wire x1="-86.36" y1="2.54" x2="-86.36" y2="15.24" width="0.1524" layer="91"/>
+<wire x1="-86.36" y1="15.24" x2="-93.98" y2="15.24" width="0.1524" layer="91"/>
+<junction x="-86.36" y="2.54"/>
+<wire x1="-93.98" y1="15.24" x2="-96.52" y2="15.24" width="0.1524" layer="91"/>
+<wire x1="-96.52" y1="15.24" x2="-96.52" y2="30.48" width="0.1524" layer="91"/>
+<pinref part="D1" gate="G$1" pin="G"/>
+<wire x1="-96.52" y1="30.48" x2="-86.36" y2="30.48" width="0.1524" layer="91"/>
+</segment>
+</net>
