File: Circuit/PCB/CANBUS_USB.brd (EAGLE design)
At the start: 71.1 x 75.9 mm, 30 parts

Commit message: update xcode
Parts:
- removed C4: 2.2uf, SparkFun-Capacitors:0603-CAP
- removed C5: 4.7uf, SparkFun-Capacitors:0603-CAP
- removed C6: 0.1uf, SparkFun-Capacitors:0603-CAP
- removed CAN_INPUT1, CAN_INPUT2: (no value), SparkFun-Connectors:JST-2-SMD
- removed D3: PESD1CAN, diode:SOT23
- removed J2, J3: (no value), SparkFun-Connectors:1X02
- removed J4: (no value), SparkFun-Connectors:1X06-1MM
- removed R7_60, R8_60: 60, SparkFun-Resistors:0603-RES
- removed R9: 10K, SparkFun-Resistors:0603-RES
- removed U$3: SN65HVD232Q, TCAN1042DRQ1:SN65HVD232Q
Connections:
- removed net CAN_H1: CAN_INPUT1.1, CAN_INPUT2.1, D3.1, J3.1, U$3.CANH
- removed net CAN_L1: CAN_INPUT1.2, CAN_INPUT2.2, D3.2, J2.2, U$3.CANL
- removed net CAN_RX: J4.4
- removed net CAN_STB: J4.5
- removed net N$13: C5.1, R7_60.1, R8_60.2
- removed net N$14: J2.1, R8_60.1
- removed net N$2: J4.6
- removed net N$5: U$3.VREF
- removed net N$6: R9.1, U$3.RS
- removed net N$7: J3.2, R7_60.2
- net 3.3V: no longer C4.1, C6.1, J4.2, U$3.VCC
- net CAN_RX3: no longer U$3.R
- net CAN_TX: no longer J4.3
- net CAN_TX3: no longer U$3.D
- net GND_MCU: no longer C4.2, C5.2, C6.2, D3.3, J4.1, R9.2, U$3.GND
Routing:
- net CAN_L1: track 43.0 -> 0.00 mm
- net CAN_H1: track 42.6 -> 0.00 mm, vias 1 -> 0
- net N$6: track 12.6 -> 0.00 mm, vias 2 -> 0
- net N$7: track 9.12 -> 0.00 mm
- net N$14: track 6.86 -> 0.00 mm
- net N$13: track 5.11 -> 0.00 mm
- net 3.3V: track 200.4 -> 197.2 mm
