File: Circuit/PCB/CANBUS_USB.sch (EAGLE design)
At the start: 22 parts

Commit message: client server
Connections:
- net KEY_03: now also R3.1; no longer R4.1
- net KEY_04: now also R4.1; no longer R3.1
Other:
- moved on the sheet: R3, R4
Changed lines of the file:
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@@
 <part name="R1" library="microbuilder" deviceset="RESISTOR" device="1206"/>
 <part name="R2" library="microbuilder" deviceset="RESISTOR" device="1206"/>
+<part name="R4" library="microbuilder" deviceset="RESISTOR" device="1206"/>
 <part name="R3" library="microbuilder" deviceset="RESISTOR" device="1206"/>
-<part name="R4" library="microbuilder" deviceset="RESISTOR" device="1206"/>
 <part name="OUT_LED_1" library="fab" deviceset="LED" device="FAB1206"/>
 <part name="OUT_LED_R1" library="fab" deviceset="RES-US" device="1206FAB" value="500"/>
@@
 <instance part="R1" gate="G$1" x="33.02" y="180.34" rot="R90"/>
 <instance part="R2" gate="G$1" x="101.6" y="180.34" rot="R90"/>
-<instance part="R3" gate="G$1" x="101.6" y="152.4" rot="R90"/>
-<instance part="R4" gate="G$1" x="33.02" y="152.4" rot="R90"/>
+<instance part="R4" gate="G$1" x="101.6" y="152.4" rot="R90"/>
+<instance part="R3" gate="G$1" x="33.02" y="152.4" rot="R90"/>
 <instance part="OUT_LED_1" gate="G$1" x="210.82" y="167.64" rot="R90"/>
 <instance part="OUT_LED_R1" gate="G$1" x="193.04" y="167.64" rot="R180"/>
@@
 </segment>
 <segment>
-<pinref part="R4" gate="G$1" pin="2"/>
+<pinref part="R3" gate="G$1" pin="2"/>
 <wire x1="33.02" y1="157.48" x2="33.02" y2="162.56" width="0.1524" layer="91"/>
 <label x="33.02" y="162.56" size="1.778" layer="95"/>
@@
 </segment>
 <segment>
-<pinref part="R3" gate="G$1" pin="2"/>
+<pinref part="R4" gate="G$1" pin="2"/>
 <wire x1="101.6" y1="157.48" x2="101.6" y2="160.02" width="0.1524" layer="91"/>
 <label x="101.6" y="162.56" size="1.778" layer="95"/>
@@
 <pinref part="S3" gate="G$1" pin="S1"/>
 <wire x1="22.86" y1="144.78" x2="33.02" y2="144.78" width="0.1524" layer="91"/>
-<pinref part="R4" gate="G$1" pin="1"/>
+<pinref part="R3" gate="G$1" pin="1"/>
 <wire x1="33.02" y1="144.78" x2="43.18" y2="144.78" width="0.1524" layer="91"/>
 <wire x1="33.02" y1="147.32" x2="33.02" y2="144.78" width="0.1524" layer="91"/>
@@
 <pinref part="S4" gate="G$1" pin="S1"/>
 <wire x1="111.76" y1="144.78" x2="101.6" y2="144.78" width="0.1524" layer="91"/>
-<pinref part="R3" gate="G$1" pin="1"/>
+<pinref part="R4" gate="G$1" pin="1"/>
 <wire x1="101.6" y1="144.78" x2="93.98" y2="144.78" width="0.1524" layer="91"/>
 <wire x1="101.6" y1="147.32" x2="101.6" y2="144.78" width="0.1524" layer="91"/>

Commit message: PCB
Parts:
- removed CAN_OUTPUT: (no value), SparkFun-Connectors:CONN_02-JST-2MM-SMT
- removed CAN_R3: 120ohm, SparkFun-Resistors:RESISTOR1206
- added CONN01, CONN03: TMMH-105-12, TMMH-105-XX-XX-DV:TMMH-105-12
- added J1: (no value), SparkFun-Connectors:CONN_06SMD-1MM
- added R5: 10k, resistor:R-US_M1206
- added SJ4: JUMPER-PAD-3-2OF3_NC_BY_TRACE_SMALL, SparkFun-Passives:JUMPER-PAD-3-2OF3_NC_BY_TRACE_SMALL
- added SJ6: A-VCC1, SparkFun-Passives:JUMPER-PAD-2-NO
Connections:
- new net GPIO_01: CONN03.1, U$1.5/PWM
- new net GPIO_02: CONN03.2, U$1.6/PWM
- new net GPIO_03: CONN03.3, U$1.7/RX3
- new net GPIO_04: CONN03.4, U$1.8/TX3
- new net GPIO_05: CONN03.5, U$1.9/RX2/PWM
- new net GPIO_06: CONN03.6, U$1.10/TX2/PWM
- new net GPIO_07: CONN03.7, U$1.11/MOSI
- new net GPIO_08: CONN03.8, U$1.12/MISO
- new net GPIO_09: CONN03.9, U$1.18/A4/T/SDA0
- new net GPIO_10: CONN03.10, U$1.19/A5/T/SCL0
- new net GPIO_11: CONN01.1, U$1.13/SCK/LED
- new net GPIO_12: CONN01.2, U$1.14/A0
- new net GPIO_13: CONN01.3, U$1.17/A3/T
- new net GPIO_14: CONN01.4, U$1.24
- new net GPIO_15: CONN01.5, U$1.25/T/PWM
- new net GPIO_16: CONN01.6, U$1.26/A15
- new net GPIO_17: CONN01.7, U$1.27/A16
- new net GPIO_18: CONN01.8, U$1.28/A17
- new net GPIO_19: CONN01.9, U$1.29/A18/SCL1
- new net GPIO_20: CONN01.10, U$1.30/A19/SDA1
- new net N$17: R5.2, SJ4.2
- new net N$20: U$1.31/A20
- new net N$22: J1.6
- net 3.3V: now also C2.2, J1.2, TCAN1042.VCC
- net CAN_H: no longer CAN_OUTPUT.2, CAN_R3.1
- net CAN_L: no longer CAN_OUTPUT.1, CAN_R3.2
- net CAN_RX: now also J1.4
- net CAN_STB: now also J1.5, SJ4.1, SJ4.3, SJ6.1, SJ6.2, U$1.2
- net CAN_TX: now also J1.3
- net GND_MCU: now also CONN01.12, CONN03.12, J1.1, R5.1
- net VCC_MCU: now also CONN01.11, CONN03.11; no longer C2.2, TCAN1042.VCC
Other:
- moved on the sheet: CAN_INPUT, CAN_R2

Commit message: components
Parts:
- removed C2, C3: 0.1uF, adafruit:C-USC1206
- removed CAN_INPUT: (no value), SparkFun-Connectors:CONN_02-JST-2MM-SMT
- removed CAN_LED: LEDFAB1206, fab:LEDFAB1206
- removed CAN_LED_R: 500, fab:RES-US1206FAB
- removed CAN_R2: 120ohm, SparkFun-Resistors:RESISTOR1206
- removed R5: 10k, resistor:R-US_M1206
- removed SJ4: JUMPER-PAD-3-2OF3_NC_BY_TRACE_SMALL, SparkFun-Passives:JUMPER-PAD-3-2OF3_NC_BY_TRACE_SMALL
- removed SJ6: A-VCC1, SparkFun-Passives:JUMPER-PAD-2-NO
- removed TCAN1042: Value, TCAN1042DRQ1:TCAN1042DRQ1
- removed U$1: TEENSY_3.1-3.2_ALL_PINS&PADS, Teensy_3_and_LC_Series_Boards_v1.4:TEENSY_3.1-3.2_ALL_PINS&PADS
- added C4: 2.2uf, SparkFun-Capacitors:0.1UF-25V(+80/-20%)(0603)
- added C5: 4.7uf, SparkFun-Capacitors:0.1UF-25V(+80/-20%)(0603)
- added C6: 0.1uf, SparkFun-Capacitors:0.1UF-25V(+80/-20%)(0603)
- added CAN_INPUT1, CAN_INPUT2: (no value), SparkFun-Connectors:CONN_02-JST-2MM-SMT
- added D3: PESD1CAN, diode:PESD1CAN
- added J2, J3: (no value), SparkFun-Connectors:CONN_02
- added J4: (no value), SparkFun-Connectors:CONN_06SMD-1MM
- added J6: (no value), SparkFun-Connectors:CONN_06NO_SILK_NO_POP
- added R7_60, R8_60: 60, SparkFun-Resistors:10KOHM-1/10W-1%(0603)0603
- added R9: 10K, SparkFun-Resistors:10KOHM-1/10W-1%(0603)0603
- added U$2: TEENSY_4.0_WITH_SMD_HEADER_PINS, Teensy4:TEENSY_4.0_WITH_SMD_HEADER_PINS
- added U$3: SN65HVD232Q, TCAN1042DRQ1:SN65HVD232Q
Connections:
- net N$22 renamed SWITCH_01
- removed net CAN_H: CAN_INPUT.2, CAN_R2.1, TCAN1042.CANH
- removed net CAN_L: CAN_INPUT.1, CAN_R2.2, TCAN1042.CANL
- removed net N$17: R5.2, SJ4.2
- removed net N$193: CAN_LED.A, CAN_LED_R.1
- removed net N$20: U$1.31/A20
- removed net VCC_MCU: C3.1, CONN01.11, CONN03.11, U$1.VUSB
- new net CAN_H1: CAN_INPUT1.2, CAN_INPUT2.2, D3.1, J3.1, U$3.CANH
- new net CAN_H2: J6.5
- new net CAN_L1: CAN_INPUT1.1, CAN_INPUT2.1, D3.2, J2.2, U$3.CANL
- new net CAN_L2: J6.6
- new net CAN_RX2: J6.4, U$2.0/RX1/T/CRX2
- new net CAN_RX3: U$2.30/CRX3, U$3.RXD
- new net CAN_TX2: J6.3, U$2.1/TX1/T/CTX2
- new net CAN_TX3: U$2.31/CTX3, U$3.TXD
- new net GPIO_SCL: CONN01.10, U$2.19/A5/SCL0
- new net GPIO_SDA: CONN01.9, U$2.18/A4/SDA0
- new net LED_IN: J1.4
- new net N$10: U$2.24/A10/SCL2
- new net N$13: C5.1, R7_60.1, R8_60.2
- new net N$14: J2.1, R8_60.1
- new net N$28: U$2.6
- new net N$5: U$3.NC
- new net N$6: R9.1, U$3.STB
- new net N$7: J3.2, R7_60.2
- new net SWITCH_02: J1.5
- net 3.3V: now also C4.1, C6.1, CONN01.11, CONN03.11, J4.2, J6.1, U$2.3.3V, U$3.VCC; no longer C2.2, TCAN1042.VCC, U$1.3.3V
- net CAN_RX: now also J4.4; no longer J1.4, TCAN1042.RXD, U$1.4/CAN-RX/PWM
- net CAN_STB: now also J4.5; no longer J1.5, SJ4.1, SJ4.3, SJ6.1, SJ6.2, TCAN1042.STB, U$1.2
- net CAN_TX: now also J4.3; no longer CAN_LED_R.2, TCAN1042.TXD, U$1.3/CAN-TX/PWM
- net GND_MCU: now also C4.2, C5.2, C6.2, D3.3, J4.1, J6.2, R9.2, U$2.GND, U$3.GND; no longer C2.1, C3.2, CAN_LED.C, R5.1, TCAN1042.GND, U$1.GND
- net GPIO_01: now also U$2.7/RX2; no longer U$1.5/PWM
- net GPIO_02: now also U$2.8/TX2; no longer U$1.6/PWM
- net GPIO_03: now also U$2.9; no longer U$1.7/RX3
- net GPIO_04: now also U$2.10/CS; no longer U$1.8/TX3
- net GPIO_05: now also U$2.11/MOSI; no longer U$1.9/RX2/PWM
- net GPIO_06: now also U$2.12/MISO; no longer U$1.10/TX2/PWM
- net GPIO_07: now also U$2.13/SCK/LED; no longer U$1.11/MOSI
- net GPIO_08: now also U$2.14/A0/TX3; no longer U$1.12/MISO
- net GPIO_09: now also U$2.17/A3/SDA1; no longer U$1.18/A4/T/SDA0
- net GPIO_10: now also U$2.26/A12/MOSI1; no longer U$1.19/A5/T/SCL0
- net GPIO_11: now also U$2.25/A11/SDA2; no longer U$1.13/SCK/LED
- net GPIO_12: now also U$2.20/A6/TX5; no longer U$1.14/A0
- net GPIO_13: now also U$2.21/A7/RX5; no longer U$1.17/A3/T
- net GPIO_14: now also U$2.22/A8/CTX1; no longer U$1.24
- net GPIO_15: now also U$2.23/A9/CRX1; no longer U$1.25/T/PWM
- net GPIO_16: now also U$2.33; no longer U$1.26/A15
- net GPIO_17: now also U$2.32; no longer U$1.27/A16
- net GPIO_18: now also U$2.29/TX7; no longer U$1.28/A17
- net GPIO_19: now also U$2.28/RX7; no longer CONN01.9, U$1.29/A18/SCL1
- net GPIO_20: now also U$2.27/A13/SCK1; no longer CONN01.10, U$1.30/A19/SDA1
- net KEY_01: now also U$2.2; no longer U$1.20/A6/PWM
- net KEY_02: now also U$2.3; no longer U$1.21/A7/PWM
- net KEY_03: now also U$2.4; no longer U$1.22/A8/T/PWM
- net KEY_04: now also U$2.5; no longer U$1.23/A9/T/PWM
- net LED_15: now also U$2.15/A1/RX3; no longer U$1.15/A1/T
- net LED_16: now also U$2.16/A2/SCL1; no longer U$1.16/A2/T
- net N$2: now also J4.6; no longer U$1.VIN
- net N$3: now also U$2.VIN; no longer TCAN1042.NC
Other:
- moved on the sheet: CONN01, CONN03, J1, OUT_LED_1, OUT_LED_2, OUT_LED_R1, OUT_LED_R2, R1, R2, R3, R4, S1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

Commit message: update xcode
Parts:
- removed C4: 2.2uf, SparkFun-Capacitors:0.1UF-25V(+80/-20%)(0603)
- removed C5: 4.7uf, SparkFun-Capacitors:0.1UF-25V(+80/-20%)(0603)
- removed C6: 0.1uf, SparkFun-Capacitors:0.1UF-25V(+80/-20%)(0603)
- removed CAN_INPUT1, CAN_INPUT2: (no value), SparkFun-Connectors:CONN_02-JST-2MM-SMT
- removed D3: PESD1CAN, diode:PESD1CAN
- removed J2, J3: (no value), SparkFun-Connectors:CONN_02
- removed J4: (no value), SparkFun-Connectors:CONN_06SMD-1MM
- removed R7_60, R8_60: 60, SparkFun-Resistors:10KOHM-1/10W-1%(0603)0603
- removed R9: 10K, SparkFun-Resistors:10KOHM-1/10W-1%(0603)0603
- removed U$3: SN65HVD232Q, TCAN1042DRQ1:SN65HVD232Q
Connections:
- removed net CAN_H1: CAN_INPUT1.2, CAN_INPUT2.2, D3.1, J3.1, U$3.CANH
- removed net CAN_L1: CAN_INPUT1.1, CAN_INPUT2.1, D3.2, J2.2, U$3.CANL
- removed net CAN_RX: J4.4
- removed net CAN_STB: J4.5
- removed net N$13: C5.1, R7_60.1, R8_60.2
- removed net N$14: J2.1, R8_60.1
- removed net N$2: J4.6
- removed net N$5: U$3.NC
- removed net N$6: R9.1, U$3.STB
- removed net N$7: J3.2, R7_60.2
- net 3.3V: no longer C4.1, C6.1, J4.2, U$3.VCC
- net CAN_RX3: no longer U$3.RXD
- net CAN_TX: no longer J4.3
- net CAN_TX3: no longer U$3.TXD
- net GND_MCU: no longer C4.2, C5.2, C6.2, D3.3, J4.1, R9.2, U$3.GND
