File: Circuit/PCB/CANBUS_USB.sch (EAGLE design)
At the start: 30 parts

Commit message: can bus
Parts:
- removed CAN_INPUT1, CAN_INPUT2: (no value), SparkFun-Connectors:CONN_02-JST-2MM-SMT
- removed J2, J3: (no value), SparkFun-Connectors:CONN_02
- removed J6: (no value), SparkFun-Connectors:CONN_06NO_SILK_NO_POP
- removed OUT_LED_1, OUT_LED_2: LEDFAB1206, fab:LEDFAB1206
- removed OUT_LED_R1, OUT_LED_R2: 500, fab:RES-US1206FAB
- removed R7_60, R8_60: 60, SparkFun-Resistors:10KOHM-1/10W-1%(0603)0603
- removed R9: 10K, SparkFun-Resistors:10KOHM-1/10W-1%(0603)0603
- removed U$3: SN65HVD232Q, TCAN1042DRQ1:SN65HVD232Q
- added C10: 0.1uf, SparkFun-Capacitors:0.1UF-25V(+80/-20%)(0603)
- added CAN_2_I, CAN_2_O, CAN_FD_I, CAN_FD_O: (no value), SparkFun-Connectors:CONN_02-JST-2MM-SMT
- added D5: PESD1CAN, diode:PESD1CAN
- added J2_FD, J3_2: (no value), SparkFun-Connectors:CONN_02
- added MCP2562, MCP2562FD: MCP2562, MCP2562:MCP2562
- added OUT_LED_3, OUT_LED_4: LEDFAB1206, fab:LEDFAB1206
- added OUT_LED_R3, OUT_LED_R4: 500, fab:RES-US1206FAB
- added R5: 120Ohms, SparkFun-Resistors:10KOHM-1/10W-1%(0603)0603
- added R8: 120Ohms FD, SparkFun-Resistors:10KOHM-1/10W-1%(0603)0603
- C4: value 2.2uf -> 0.1uf
- C5: value 4.7uf -> 0.1uf
- CONN01, CONN03: value TMMH-105-12 -> 2X6 FEMALE; device TMMH-105-XX-XX-DV:TMMH-105-12 -> SparkFun-Connectors:CONN_06X2PTH_FEMALE
Connections:
- removed net CAN_H2: J6.5
- removed net CAN_L2: J6.6
- removed net CAN_RX: J4.4
- removed net CAN_STB: J4.5
- removed net CAN_TX: J1.3, J4.3
- removed net LED_IN: J1.4
- removed net N$1: OUT_LED_2.A, OUT_LED_R2.1
- removed net N$10: U$2.24/A10/SCL2
- removed net N$13: C5.1, R7_60.1, R8_60.2
- removed net N$14: J2.1, R8_60.1
- removed net N$28: U$2.6
- removed net N$3: U$2.VIN
- removed net N$4: OUT_LED_1.A, OUT_LED_R1.1
- new net CAN_H: CAN_FD_I.2, CAN_FD_O.2, D3.1, MCP2562FD.CANH, R8.1
- new net CAN_L: CAN_FD_I.1, CAN_FD_O.1, D3.2, J2_FD.2, MCP2562FD.CANL
- new net VCC_5V: C10.1, C4.1, CONN01.11, CONN03.11, J4.2, MCP2562.VDD, MCP2562FD.VDD, U$2.VIN
- net 3.3V: now also C5.1, CONN01.9, CONN03.9, MCP2562.VIO, MCP2562FD.VIO; no longer C4.1, CONN01.11, CONN03.11, J4.2, J6.1, U$3.VCC
- net CAN_H1: now also CAN_2_I.2, CAN_2_O.2, D5.1, MCP2562.CANH, R5.1; no longer CAN_INPUT1.2, CAN_INPUT2.2, D3.1, J3.1, U$3.CANH
- net CAN_L1: now also CAN_2_I.1, CAN_2_O.1, D5.2, J3_2.2, MCP2562.CANL; no longer CAN_INPUT1.1, CAN_INPUT2.1, D3.2, J2.2, U$3.CANL
- net CAN_RX2: now also CONN01.3, MCP2562.RXD; no longer J6.4
- net CAN_RX3: now also MCP2562FD.RXD; no longer U$3.RXD
- net CAN_TX2: now also CONN01.4, MCP2562.TXD; no longer J6.3
- net CAN_TX3: now also MCP2562FD.TXD; no longer U$3.TXD
- net GND_MCU: now also C10.2, CONN01.10, CONN03.10, D5.3, MCP2562.STBY, MCP2562.VSS, MCP2562FD.STBY, MCP2562FD.VSS, OUT_LED_3.C, OUT_LED_4.C; no longer J6.2, OUT_LED_1.C, OUT_LED_2.C, R9.2, U$3.GND
- net GPIO_01: now also CONN03.3, U$2.2; no longer CONN03.1, U$2.7/RX2
- net GPIO_02: now also CONN03.4, U$2.3; no longer CONN03.2, U$2.8/TX2
- net GPIO_03: now also CONN03.5, U$2.4; no longer CONN03.3, U$2.9
- net GPIO_04: now also CONN01.5; no longer CONN03.4
- net GPIO_05: now also CONN01.6; no longer CONN03.5
- net GPIO_06: now also CONN01.7; no longer CONN03.6
- net GPIO_07: now also CONN03.8; no longer CONN03.7
- net GPIO_08: now also CONN01.8; no longer CONN03.8
- net GPIO_09: now also U$2.15/A1/RX3; no longer CONN03.9, U$2.17/A3/SDA1
- net GPIO_10: now also CONN03.1, U$2.16/A2/SCL1; no longer CONN03.10, U$2.26/A12/MOSI1
- net GPIO_11: now also CONN03.2, U$2.17/A3/SDA1; no longer CONN01.1, U$2.25/A11/SDA2
- net GPIO_12: now also J1.3; no longer CONN01.2
- net GPIO_13: now also J1.4; no longer CONN01.3
- net GPIO_14: now also CONN03.7, U$2.25/A11/SDA2; no longer CONN01.4, U$2.22/A8/CTX1
- net GPIO_15: now also J4.3, U$2.26/A12/MOSI1; no longer CONN01.5, U$2.23/A9/CRX1
- net GPIO_16: now also J4.4, U$2.27/A13/SCK1; no longer CONN01.6, U$2.33
- net GPIO_17: now also J4.5, U$2.28/RX7; no longer CONN01.7, U$2.32
- net GPIO_18: now also J4.6; no longer CONN01.8
- net GPIO_19: now also U$2.32; no longer U$2.28/RX7
- net GPIO_20: now also CONN03.6, U$2.24/A10/SCL2; no longer U$2.27/A13/SCK1
- net GPIO_SCL: now also CONN01.1; no longer CONN01.10
- net GPIO_SDA: now also CONN01.2; no longer CONN01.9
- net KEY_01: now also U$2.6; no longer U$2.2
- net KEY_02: now also U$2.7/RX2; no longer U$2.3
- net KEY_03: now also U$2.8/TX2; no longer U$2.4
- net KEY_04: now also U$2.9; no longer U$2.5
- net LED_15: now also OUT_LED_R4.2, U$2.22/A8/CTX1; no longer OUT_LED_R1.2, U$2.15/A1/RX3
- net LED_16: now also OUT_LED_R3.2, U$2.23/A9/CRX1; no longer OUT_LED_R2.2, U$2.16/A2/SCL1
- net N$2: now also J2_FD.1, R8.2; no longer J4.6
- net N$5: now also J3_2.1, R5.2; no longer U$3.NC
- net N$6: now also OUT_LED_3.A, OUT_LED_R3.1; no longer R9.1, U$3.STB
- net N$7: now also OUT_LED_4.A, OUT_LED_R4.1; no longer J3.2, R7_60.2
- net SWITCH_01: now also U$2.5
- net SWITCH_02: now also U$2.33
Other:
- moved on the sheet: C4, C5, C6, CONN01, CONN03, D3, J1, J4
