File: Circuit/PCB/teensyMotors02_upSwitch_LED_SX.sch (EAGLE design)
At the start: 65 parts, among them SW1 219-10, SW2 B3F-1000, SW3 B3F-1000, SW4 B3F-1000, SW5 B3F-1000, SW6 B3F-1000, SW7 B3F-1000, SW8 B3F-1000, SW9 B3F-1000

Commit message: board
Parts:
- CONN01, CONN02: value TMMH-105-12 -> 2X6 FEMALE; device TMMH-105-XX-XX-DV:TMMH-105-12 -> SparkFun-Connectors:CONN_06X2PTH_FEMALE
- U$1, U$2, U$3: value SX1509 -> SX1509HOLE; device SX1509_s:SX1509 -> SX1509_s:SX1509HOLE
Connections:
- new net N$1: S1.7
Other:
- moved on the sheet: CONN01, CONN02

Commit message: circuit up
Connections:
- net VCC_5V: now also S1.8; no longer S1.2
Changed lines of the file:
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@@
 <clearance class="1" value="0.2"/>
 </class>
-<class number="4" name="5v" width="0.35" drill="0">
+<class number="2" name="3v" width="0.45" drill="0">
+<clearance class="2" value="0.2"/>
+</class>
+<class number="4" name="5v" width="0.45" drill="0">
 <clearance class="4" value="0.2"/>
 </class>
@@
 <part name="JP3" library="microbuilder" deviceset="HEADER-1X4" device="ROUND"/>
 <part name="S1" library="JS207011SCQNR" deviceset="JS207011SCQNR" device=""/>
-<part name="U$1" library="SX1509_s" deviceset="SX1509" device="HOLE" value="SX1509HOLE"/>
-<part name="U$2" library="SX1509_s" deviceset="SX1509" device="HOLE" value="SX1509HOLE"/>
-<part name="U$3" library="SX1509_s" deviceset="SX1509" device="HOLE" value="SX1509HOLE"/>
+<part name="U$1" library="SX1509_s" deviceset="SX1509" device="HOLE" package3d_urn="urn:adsk.eagle:package:19026190/1" value="SX1509HOLE"/>
+<part name="U$2" library="SX1509_s" deviceset="SX1509" device="HOLE" package3d_urn="urn:adsk.eagle:package:19026190/1" value="SX1509HOLE"/>
+<part name="U$3" library="SX1509_s" deviceset="SX1509" device="HOLE" package3d_urn="urn:adsk.eagle:package:19026190/1" value="SX1509HOLE"/>
 <part name="SW2" library="Switch" library_urn="urn:adsk.eagle:library:11396471" deviceset="B3F-1000" device="" package3d_urn="urn:adsk.eagle:package:10899221/2"/>
 <part name="SW3" library="Switch" library_urn="urn:adsk.eagle:library:11396471" deviceset="B3F-1000" device="" package3d_urn="urn:adsk.eagle:package:10899221/2"/>
@@
 </segment>
 </net>
-<net name="3.3V" class="0">
+<net name="3.3V" class="2">
 <segment>
 <wire x1="35.56" y1="147.32" x2="27.94" y2="147.32" width="0.1524" layer="91"/>
@@
 </segment>
 <segment>
-<pinref part="S1" gate="G$1" pin="2"/>
-<wire x1="165.1" y1="167.64" x2="172.72" y2="167.64" width="0.1524" layer="91"/>
-<label x="172.72" y="167.64" size="1.016" layer="95" xref="yes"/>
+<pinref part="S1" gate="G$1" pin="8"/>
+<wire x1="165.1" y1="160.02" x2="170.18" y2="160.02" width="0.1524" layer="91"/>
+<label x="170.18" y="160.02" size="1.016" layer="95" xref="yes"/>
 </segment>
 </net>
@@
 <pinref part="S1" gate="G$1" pin="3"/>
 <wire x1="149.86" y1="167.64" x2="144.78" y2="167.64" width="0.1524" layer="91"/>
-<label x="144.78" y="165.1" size="1.016" layer="95" rot="R180" xref="yes"/>
-</segment>
-</net>
+<label x="144.78" y="167.64" size="1.016" layer="95" rot="R180" xref="yes"/>
+</segment>
+</net>
