File: Circuit/PCB/teensyMotors02_upSwitch_LED_SX.brd (EAGLE design)
At the start: 72 x 150.1 mm, 65 parts, among them SW1 219-10, SW2 B3F-1000, SW3 B3F-1000, SW4 B3F-1000, SW5 B3F-1000, SW6 B3F-1000, SW7 B3F-1000, SW8 B3F-1000, SW9 B3F-1000

Commit message: board
Parts:
- CONN01, CONN02: value TMMH-105-12 -> 2X6 FEMALE; device TMMH-105-XX-XX-DV:TMMH-105-12 -> SparkFun-Connectors:2X6
- U$1, U$2, U$3: value SX1509 -> SX1509HOLE; device SX1509_s:SX1509 -> SX1509_s:SX1509_HOLE
- moved JP3 12.2 mm to (16.2, 115.3), turned to 90 degrees
- moved JP2 11.0 mm to (14.9, 122.1)
- moved R15 7.72 mm to (48.2, 47.8)
- moved R29 7.72 mm to (45.7, 47.8)
- moved R30 7.72 mm to (43.1, 47.8)
- moved R31 7.72 mm to (40.5, 47.8)
- moved R32 7.72 mm to (38.0, 47.8)
- moved R33 7.72 mm to (35.4, 47.8)
- moved R34 7.72 mm to (32.9, 47.8)
- moved R35 7.72 mm to (30.3, 47.8)
- moved R36 7.72 mm to (27.8, 47.8)
- moved R37 7.72 mm to (25.2, 47.8)
- moved CONN02 6.16 mm to (66.5, 122.4)
- moved CONN01 6.14 mm to (8.61, 122.4)
- moved SW1 4.32 mm to (36.3, 36.5)
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Connections:
- new net N$1: S1.7
- net 3.3V: now also U$1.3.3V_2, U$2.3.3V_2, U$3.3.3V_2; no longer U$1.3.3V_1, U$2.3.3V_1, U$3.3.3V_1
Routing:
- net 3.3V: track 422.2 -> 484.4 mm, vias 7 -> 4
- net GND_MCU: track 627.8 -> 674.4 mm, vias 31 -> 25
- net SCL_00: track 248.3 -> 285.8 mm, vias 16 -> 2
- net NEOPIXEL_04: track 92.4 -> 122.2 mm, vias 5 -> 4
- net 10_SX2: track 33.2 -> 60.5 mm, vias 1 -> 2
- net 12_SX1: track 89.3 -> 65.7 mm, vias 3 -> 4
- net 3_SX2: track 33.7 -> 55.1 mm, vias 1 -> 0
- net INT_01: track 63.6 -> 43.3 mm, vias 2 -> 0
- net 12_SX2: track 42.9 -> 60.1 mm
- net CAN_TX2: track 29.0 -> 15.1 mm
- net 4_SX2: track 40.4 -> 52.7 mm, vias 1 -> 0
- net 11_SX2: track 33.5 -> 43.8 mm
- net CAN_RX2: track 23.2 -> 13.7 mm
- net 15_SX2: track 74.1 -> 83.0 mm, vias 3 -> 0
- net 6_SX2: track 72.2 -> 63.6 mm
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Other:
- outline, holes or cut-outs redrawn
- board text added: "-"
- board text added: "0"
- board text added: "3.3V"
- board text added: "GND"
- board text added: "Power"
- board text removed: "8"

Commit message: merge
Routing:
- net NEOPIXEL_04: track 122.2 -> 100.4 mm
- net GND_MCU: track 674.4 -> 667.5 mm
- net N$193: track 5.36 -> 4.27 mm

Commit message: circuit up
Parts:
- moved U$2 3.24 mm to (38.1, 117.7), flipped to the top
- moved U$3 3.10 mm to (38.1, 35.6), flipped to the top
- moved U$1 2.54 mm to (37.6, 75.8), flipped to the top
- moved SW1 1.15 mm to (37.1, 35.7)
- moved R15 0.49 mm to (48.3, 48.3)
- moved R29 0.49 mm to (45.7, 48.3)
- moved R30 0.49 mm to (43.2, 48.3)
- moved R31 0.49 mm to (40.6, 48.3)
- moved R32 0.49 mm to (38.1, 48.3)
- moved R33 0.49 mm to (35.5, 48.3)
- moved R34 0.49 mm to (33.0, 48.3)
- moved R35 0.49 mm to (30.4, 48.3)
- moved R36 0.49 mm to (27.9, 48.3)
- moved R37 0.49 mm to (25.3, 48.3)
- moved JP2 0.35 mm to (14.8, 122.5)
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Connections:
- net VCC_5V: now also S1.8; no longer S1.2
Routing:
- net 10_SX1: track 74.8 -> 136.5 mm, vias 1 -> 2
- net 3.3V: track 484.1 -> 426.7 mm, vias 4 -> 0
- net 2_SX1: track 70.9 -> 118.4 mm, vias 2 -> 4
- net 4_SX1: track 83.4 -> 128.7 mm, vias 2 -> 4
- net 8_SX1: track 63.3 -> 105.8 mm, vias 1 -> 2
- net SCL_00: track 285.8 -> 243.5 mm
- net 6_SX3: track 15.7 -> 56.7 mm, vias 0 -> 5
- net INT_02: track 14.3 -> 55.0 mm
- net 8_SX3: track 24.6 -> 62.5 mm, vias 0 -> 4
- net GND_MCU: track 667.5 -> 705.0 mm, vias 25 -> 41
- net 3_SX1: track 74.0 -> 110.4 mm, vias 4 -> 3
- net 14_SX3: track 22.1 -> 55.9 mm, vias 0 -> 3
- net NEOPIXEL_03: track 69.5 -> 103.0 mm, vias 1 -> 3
- net 14_SX1: track 68.1 -> 35.3 mm
- net 14_SX2: track 74.3 -> 45.9 mm
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
Commit message: update circuit sx
Routing:
- net NEOPIXEL_04: track 97.0 -> 100.5 mm
- net 6_SX1: track 127.1 -> 130.5 mm
- net 4_SX3: track 79.8 -> 83.0 mm
- net INT_01: track 71.5 -> 74.7 mm
- net 13_SX3: track 41.2 -> 42.7 mm
- net 3_SX3: track 98.7 -> 100.1 mm
- net 12_SX1: track 67.8 -> 69.1 mm
- net 3.3V: track 426.7 -> 425.4 mm
- net 2_SX1: track 118.4 -> 119.6 mm
- net SCL_00: track 243.5 -> 244.6 mm
- net SDA_00: track 245.1 -> 246.1 mm
- net 7_SX1: track 49.2 -> 50.2 mm
- net 8_SX3: track 62.5 -> 63.1 mm
- net 8_SX1: track 105.8 -> 106.3 mm
- net GND_MCU: track 705.0 -> 704.8 mm, vias 41 -> 53

Commit message: return to previous pcb design
Routing:
- net NEOPIXEL_04: track 100.5 -> 97.0 mm
- net 6_SX1: track 130.5 -> 127.1 mm
- net 4_SX3: track 83.0 -> 79.8 mm
- net INT_01: track 74.7 -> 71.5 mm
- net 13_SX3: track 42.7 -> 41.2 mm
- net 3_SX3: track 100.1 -> 98.7 mm
- net 12_SX1: track 69.1 -> 67.8 mm
- net 3.3V: track 425.4 -> 426.7 mm
- net 2_SX1: track 119.6 -> 118.4 mm
- net SCL_00: track 244.6 -> 243.5 mm
- net SDA_00: track 246.1 -> 245.1 mm
- net 7_SX1: track 50.2 -> 49.2 mm
- net 8_SX3: track 63.1 -> 62.5 mm
- net 8_SX1: track 106.3 -> 105.8 mm
- net GND_MCU: track 704.8 -> 705.0 mm, vias 53 -> 41
